Commit message: working trellis

File: simple_urdf_scenes/basement_test/basement_test.urdf (robot description, URDF)
Before this commit: robot Scene, 100 links, 99 joints
Links:
- link drawer_0.477_0.177_0.533_object_8_drawer_0_0: mass 0.09999999999999999 -> 0.09999999999999998
- link drawer_0.481_0.206_0.542_object_29_drawer_0_0: mass 0.09999999999999999 -> 0.09999999999999998
- link drawer_0.496_0.171_0.531_object_9_drawer_0_0: mass 0.09999999999999999 -> 0.09999999999999998
- link drawer_0.496_0.183_0.557_object_28_drawer_0_0: mass 0.09999999999999999 -> 0.09999999999999998
- link drawer_0.506_0.185_0.545_object_7_drawer_0_0: mass 0.09999999999999999 -> 0.09999999999999998
- link drawer_0.800_0.258_0.558_object_21_drawer_0_0: mass 0.1 -> 0.10000000000000003
Joints:
- joint upper_left_cabinet_0.017_0.929_0.471_object_19_world_fixed_joint: origin xyz=4.228767027523136 -0.579342532468629 0.8417438520603431 rpy=0.0 -0.0 -1.5707963267948966 -> xyz=4.228767027523136 -0.5793425324686289 0.8417438520603431 rpy=0.0 -0.0 -1.5707963267948966
- joint upper_left_cabinet_0.279_0.929_0.299_object_18_world_fixed_joint: origin xyz=4.049086354776554 -0.08368340224450199 0.8417438520603431 rpy=0.0 -0.0 -0.7853981633974484 -> xyz=4.049086354776553 -0.08368340224450188 0.8417438520603431 rpy=0.0 -0.0 -0.7853981633974484
- joint upper_right_cabinet_0.037_0.938_0.459_object_20_world_fixed_joint: origin xyz=4.228767027523135 -1.04424492612125 0.8417438520603431 rpy=0.0 -0.0 -1.5707963267948966 -> xyz=4.228767027523136 -1.0442449261212499 0.8417438520603431 rpy=0.0 -0.0 -1.5707963267948966

Commit message: mesh generation + base_cabinet_test

File: simple_urdf_scenes/basement_test/basement_test.urdf (robot description, URDF)
Before this commit: robot Scene, 100 links, 99 joints
Links:
- link drawer_0.477_0.177_0.533_object_8_drawer_0_0: mass 0.09999999999999998 -> 0.09999999999999999
- link drawer_0.481_0.206_0.542_object_29_drawer_0_0: mass 0.09999999999999998 -> 0.09999999999999999
- link drawer_0.496_0.171_0.531_object_9_drawer_0_0: mass 0.09999999999999998 -> 0.09999999999999999
- link drawer_0.496_0.183_0.557_object_28_drawer_0_0: mass 0.09999999999999998 -> 0.09999999999999999
- link drawer_0.506_0.185_0.545_object_7_drawer_0_0: mass 0.09999999999999998 -> 0.09999999999999999
- link drawer_0.800_0.258_0.558_object_21_drawer_0_0: mass 0.10000000000000003 -> 0.1
Joints:
- joint upper_left_cabinet_0.017_0.929_0.471_object_19_world_fixed_joint: origin xyz=4.228767027523136 -0.5793425324686289 0.8417438520603431 rpy=0.0 -0.0 -1.5707963267948966 -> xyz=4.228767027523136 -0.579342532468629 0.8417438520603431 rpy=0.0 -0.0 -1.5707963267948966
- joint upper_left_cabinet_0.279_0.929_0.299_object_18_world_fixed_joint: origin xyz=4.049086354776553 -0.08368340224450188 0.8417438520603431 rpy=0.0 -0.0 -0.7853981633974484 -> xyz=4.049086354776554 -0.08368340224450199 0.8417438520603431 rpy=0.0 -0.0 -0.7853981633974484
- joint upper_right_cabinet_0.037_0.938_0.459_object_20_world_fixed_joint: origin xyz=4.228767027523136 -1.0442449261212499 0.8417438520603431 rpy=0.0 -0.0 -1.5707963267948966 -> xyz=4.228767027523135 -1.04424492612125 0.8417438520603431 rpy=0.0 -0.0 -1.5707963267948966
