Commit message: basement test run

File: simple_urdf_scenes/basement_test/basement_test.urdf (robot description, URDF)
Before this commit: robot Scene, 100 links, 99 joints
Links:
- link box_31_to_32: mass 0.06786404614499339 -> 0.06900006817694337; geometry collision box size=0.5874124768261367 0.5583849458699577 0.2103645966104818; visual box size=0.5874124768261367 0.5583849458699577 0.2103645966104818
- link box_32_to_31: mass 0.06447604599434453 -> 0.06551016250437156; geometry collision box size=0.5823849458699577 0.5634124768261367 0.19965126955854517; visual box size=0.5823849458699577 0.5634124768261367 0.19965126955854517
- link drawer_0.407_0.197_0.530_object_30_corpus: mass 0.01368820691398069 -> 0.01390375829718237; geometry collision box size=0.02 0.5183849458699576 0.1903645966104818; collision box size=0.02 0.5183849458699576 0.1903645966104818
- link drawer_0.407_0.197_0.530_object_30_drawer_0_0: geometry collision box size=0.005 0.4595464512829619 0.16036459661048177; collision box size=0.005 0.4595464512829619 0.16036459661048177
- link drawer_0.424_0.224_0.569_object_31_corpus: mass 0.01368820691398069 -> 0.01390375829718237; geometry collision box size=0.02 0.5183849458699576 0.1903645966104818; collision box size=0.02 0.5183849458699576 0.1903645966104818
- link drawer_0.424_0.224_0.569_object_31_drawer_0_0: geometry collision box size=0.005 0.4595464512829619 0.16036459661048177; collision box size=0.005 0.4595464512829619 0.16036459661048177
- link drawer_0.481_0.206_0.542_object_29_corpus: mass 0.014568915130955953 -> 0.014485445873642913; geometry collision box size=0.02 0.5183849458699576 0.16455854348159812; collision box size=0.02 0.5183849458699576 0.16455854348159812
- link drawer_0.481_0.206_0.542_object_29_drawer_0_0: mass 0.09999999999999999 -> 0.10000000000000002; geometry collision box size=0.005 0.4595464512829619 0.1345585434815981; collision box size=0.005 0.4595464512829619 0.1345585434815981
- link drawer_0.490_0.279_0.528_object_10_corpus: mass 0.01695753108153103 -> 0.017384329686903868; geometry collision box size=0.02 0.5016032887010252 0.2587573041044384; collision box size=0.02 0.5016032887010252 0.2587573041044384
- link drawer_0.490_0.279_0.528_object_10_drawer_0_0: mass 0.10000000000000002 -> 0.09999999999999999; geometry collision box size=0.005 0.4444429598309227 0.22875730410443842; collision box size=0.005 0.4444429598309227 0.22875730410443842
- link drawer_0.496_0.183_0.557_object_28_corpus: mass 0.014568915130955953 -> 0.014485445873642913; geometry collision box size=0.02 0.5183849458699576 0.16455854348159812; collision box size=0.02 0.5183849458699576 0.16455854348159812
- link drawer_0.496_0.183_0.557_object_28_drawer_0_0: mass 0.09999999999999999 -> 0.10000000000000002; geometry collision box size=0.005 0.4595464512829619 0.1345585434815981; collision box size=0.005 0.4595464512829619 0.1345585434815981
- link lower_left_cabinet_0.027_0.559_0.479_object_26_corpus: mass 0.031683652908846796 -> 0.029311895682723108; geometry collision box size=0.02 0.5234124768261367 0.540508725126398; collision box size=0.02 0.5234124768261367 0.540508725126398
- link lower_left_cabinet_0.027_0.559_0.479_object_26_door_0_0: mass 0.09999999999999999 -> 0.1; geometry collision box size=0.013999999999999999 0.04 0.024; collision box size=0.013999999999999999 0.04 0.024
- link lower_left_cabinet_0.410_0.554_0.009_object_24_corpus: mass 0.027846757352023854 -> 0.026024030286546092; geometry collision box size=0.02 0.5183849458699576 0.540508725126398; collision box size=0.02 0.5183849458699576 0.540508725126398
- link lower_left_cabinet_0.410_0.554_0.009_object_24_door_0_0: mass 0.10000000000000002 -> 0.09999999999999999; geometry collision box size=0.013999999999999999 0.04 0.024; collision box size=0.013999999999999999 0.04 0.024
- link lower_left_cabinet_0.470_0.567_0.015_object_22_corpus: mass 0.030361280693215927 -> 0.028047799178453056; geometry collision box size=0.02 0.5183849458699576 0.540508725126398; collision box size=0.02 0.5183849458699576 0.540508725126398
- link lower_left_cabinet_0.470_0.567_0.015_object_22_door_0_0: geometry collision box size=0.013999999999999999 0.04 0.024; collision box size=0.013999999999999999 0.04 0.024
- link lower_left_cabinet_0.477_0.710_0.022_object_1_corpus: mass 0.02981085749754564 -> 0.03193354675759193; geometry collision box size=0.02 0.5016032887010252 0.6940166675087931; collision box size=0.02 0.5016032887010252 0.6940166675087931
- link lower_left_cabinet_0.477_0.710_0.022_object_1_door_0_0: mass 0.10000000000000002 -> 0.09999999999999999; geometry collision box size=0.013999999999999999 0.04 0.024; collision box size=0.013999999999999999 0.04 0.024
- link lower_left_cabinet_0.481_0.705_0.014_object_5_corpus: mass 0.029964412847163186 -> 0.03265657714145913; geometry collision box size=0.02 0.5016032887010252 0.6940166675087931; collision box size=0.02 0.5016032887010252 0.6940166675087931
- link lower_left_cabinet_0.481_0.705_0.014_object_5_door_0_0: mass 0.1 -> 0.09999999999999999; geometry collision box size=0.013999999999999999 0.04 0.024; collision box size=0.013999999999999999 0.04 0.024
- link lower_left_cabinet_0.528_0.723_0.034_object_3_corpus: mass 0.03174171724556918 -> 0.034091712576451036; geometry collision box size=0.02 0.5016032887010252 0.6940166675087931; collision box size=0.02 0.5016032887010252 0.6940166675087931
- link lower_left_cabinet_0.528_0.723_0.034_object_3_door_0_0: mass 0.1 -> 0.09999999999999999; geometry collision box size=0.013999999999999999 0.04 0.024; collision box size=0.013999999999999999 0.04 0.024
- link lower_right_cabinet_0.016_0.561_0.478_object_27_corpus: mass 0.031683652908846796 -> 0.029311895682723108; geometry collision box size=0.02 0.5234124768261367 0.540508725126398; collision box size=0.02 0.5234124768261367 0.540508725126398
- link lower_right_cabinet_0.016_0.561_0.478_object_27_door_0_0: mass 0.09999999999999999 -> 0.1; geometry collision box size=0.013999999999999999 0.04 0.024; collision box size=0.013999999999999999 0.04 0.024
- link lower_right_cabinet_0.398_0.559_0.010_object_25_corpus: mass 0.027846757352023854 -> 0.026024030286546092; geometry collision box size=0.02 0.5183849458699576 0.540508725126398; collision box size=0.02 0.5183849458699576 0.540508725126398
- link lower_right_cabinet_0.398_0.559_0.010_object_25_door_0_0: mass 0.10000000000000002 -> 0.09999999999999999; geometry collision box size=0.013999999999999999 0.04 0.024; collision box size=0.013999999999999999 0.04 0.024
- link lower_right_cabinet_0.470_0.563_0.008_object_23_corpus: mass 0.030362552822140128 -> 0.028047799178453056; geometry collision box size=0.02 0.5183849458699576 0.540508725126398; collision box size=0.02 0.5183849458699576 0.540508725126398
- link lower_right_cabinet_0.470_0.563_0.008_object_23_door_0_0: geometry collision box size=0.013999999999999999 0.04 0.024; collision box size=0.013999999999999999 0.04 0.024
- link lower_right_cabinet_0.473_0.709_0.023_object_2_corpus: mass 0.02966772099081996 -> 0.03193354675759193; geometry collision box size=0.02 0.5016032887010252 0.6940166675087931; collision box size=0.02 0.5016032887010252 0.6940166675087931
- link lower_right_cabinet_0.473_0.709_0.023_object_2_door_0_0: mass 0.1 -> 0.09999999999999999; geometry collision box size=0.013999999999999999 0.04 0.024; collision box size=0.013999999999999999 0.04 0.024
- link lower_right_cabinet_0.479_0.713_0.016_object_6_corpus: mass 0.029890868390427632 -> 0.03265657714145913; geometry collision box size=0.02 0.5016032887010252 0.6940166675087931; collision box size=0.02 0.5016032887010252 0.6940166675087931
- link lower_right_cabinet_0.479_0.713_0.016_object_6_door_0_0: mass 0.1 -> 0.09999999999999999; geometry collision box size=0.013999999999999999 0.04 0.024; collision box size=0.013999999999999999 0.04 0.024
- link lower_right_cabinet_0.509_0.725_0.023_object_4_corpus: mass 0.03103085596285733 -> 0.03265657714145913; geometry collision box size=0.02 0.5016032887010252 0.6940166675087931; collision box size=0.02 0.5016032887010252 0.6940166675087931
- link lower_right_cabinet_0.509_0.725_0.023_object_4_door_0_0: mass 0.1 -> 0.09999999999999999; geometry collision box size=0.013999999999999999 0.04 0.024; collision box size=0.013999999999999999 0.04 0.024
- link upper_left_cabinet_0.392_0.934_0.031_object_12_corpus: mass 0.015984340942098114 -> 0.016226996349533968; geometry collision box size=0.01 0.3674562003068511 0.9222836146116198; collision box size=0.01 0.3674562003068511 0.9222836146116198
- link upper_left_cabinet_0.392_0.934_0.031_object_12_door_0_0: mass 0.1 -> 0.09999999999999999; geometry collision box size=0.013999999999999999 0.04 0.024; collision box size=0.013999999999999999 0.04 0.024
- link upper_right_cabinet_0.037_0.938_0.459_object_20_corpus: mass 0.01875480448505188 -> 0.019039272062411357; geometry collision box size=0.01 0.3996191792464823 0.9222836146116198; collision box size=0.01 0.3996191792464823 0.9222836146116198
- link upper_right_cabinet_0.037_0.938_0.459_object_20_door_0_0: mass 0.10000000000000002 -> 0.10000000000000003; geometry collision box size=0.013999999999999999 0.04 0.024; collision box size=0.013999999999999999 0.04 0.024
- link upper_right_cabinet_0.399_0.929_0.019_object_17_corpus: mass 0.016144343124143395 -> 0.0160072568311476; geometry collision box size=0.01 0.3674562003068511 0.9222836146116198; collision box size=0.01 0.3674562003068511 0.9222836146116198
- link upper_right_cabinet_0.399_0.929_0.019_object_17_door_0_0: mass 0.1 -> 0.10000000000000002; geometry collision box size=0.013999999999999999 0.04 0.024; collision box size=0.013999999999999999 0.04 0.024
- link upper_right_cabinet_0.483_0.931_0.019_object_15_corpus: mass 0.018155989444899975 -> 0.018155688510911403; geometry collision box size=0.01 0.3674562003068511 0.9222836146116198; collision box size=0.01 0.3674562003068511 0.9222836146116198
- link upper_right_cabinet_0.483_0.931_0.019_object_15_door_0_0: mass 0.1 -> 0.09999999999999999; geometry collision box size=0.013999999999999999 0.04 0.024; collision box size=0.013999999999999999 0.04 0.024
Joints:
- joint box_31_to_32_world_fixed_joint: origin xyz=4.135870378733311 -0.00379418384499447 0.4378816373895142 rpy=0.0 -0.0 0.0 -> xyz=4.0940938331111445 -0.008390828584466214 0.3611513574293571 rpy=0.0 -0.0 0.0
- joint box_32_to_31_world_fixed_joint: origin xyz=4.16187037873331 -0.029794183844994437 0.4325249738635459 rpy=0.0 -0.0 -1.5707963267948966 -> xyz=4.120093833111143 -0.03439082858446618 0.3557946939033888 rpy=0.0 -0.0 -1.5707963267948966
- joint drawer_0.407_0.197_0.530_object_30_corpus_to_drawer_0_0: limit lower=0.0 upper=0.42864524167672147 effort=1000.0 velocity=1.0 -> lower=0.0 upper=0.43609180615466575 effort=1000.0 velocity=1.0; origin xyz=0.0 -0.2545958281955071 0.10518229830524091 rpy=0.0 -0.0 0.0 -> xyz=0.0 -0.2591924729349788 0.10518229830524091 rpy=0.0 -0.0 0.0
- joint drawer_0.407_0.197_0.530_object_30_world_fixed_joint: origin xyz=3.2184635266508304 -0.00379418384499447 0.3326993390842733 rpy=0.0 -0.0 0.0 -> xyz=3.1766869810286638 -0.008390828584466214 0.2559690591241162 rpy=0.0 -0.0 0.0
- joint drawer_0.424_0.224_0.569_object_31_corpus_to_drawer_0_0: limit lower=0.0 upper=0.42864524167672147 effort=1000.0 velocity=1.0 -> lower=0.0 upper=0.43609180615466575 effort=1000.0 velocity=1.0; origin xyz=0.0 -0.2545958281955071 0.10518229830524091 rpy=0.0 -0.0 0.0 -> xyz=0.0 -0.2591924729349788 0.10518229830524091 rpy=0.0 -0.0 0.0
- joint drawer_0.424_0.224_0.569_object_31_world_fixed_joint: origin xyz=3.634263935763772 -0.00379418384499447 0.3326993390842733 rpy=0.0 -0.0 0.0 -> xyz=3.5924873901416055 -0.008390828584466214 0.2559690591241162 rpy=0.0 -0.0 0.0
- joint drawer_0.481_0.206_0.542_object_29_corpus_to_drawer_0_0: limit lower=0.0 upper=0.42249866384783047 effort=1000.0 velocity=1.0 -> lower=0.0 upper=0.43609180615466575 effort=1000.0 velocity=1.0; origin xyz=0.0 -0.2508016443505126 0.09227927174079907 rpy=0.0 -0.0 0.0 -> xyz=0.0 -0.2591924729349788 0.09227927174079907 rpy=0.0 -0.0 0.0
- joint drawer_0.481_0.206_0.542_object_29_world_fixed_joint: origin xyz=2.764966080413548 0.0 0.358505392213157 rpy=0.0 -0.0 0.0 -> xyz=2.733633671196923 -0.008390828584466214 0.2817751122529999 rpy=0.0 -0.0 0.0
- joint drawer_0.490_0.279_0.528_object_10_corpus_to_drawer_0_0: limit lower=0.0 upper=0.4114417491162945 effort=1000.0 velocity=1.0 -> lower=0.0 upper=0.42249866384783047 effort=1000.0 velocity=1.0; origin xyz=0.0 -0.24397638834339166 0.13937865205221922 rpy=0.0 -0.0 0.0 -> xyz=0.0 -0.2508016443505126 0.13937865205221922 rpy=0.0 -0.0 0.0
- joint drawer_0.490_0.279_0.528_object_10_world_fixed_joint: origin xyz=0.0005625013010401025 0.006825256007120972 -0.27875730410443844 rpy=0.0 -0.0 0.0 -> xyz=0.0 0.0 -0.27875730410443844 rpy=0.0 -0.0 0.0
- joint drawer_0.496_0.183_0.557_object_28_corpus_to_drawer_0_0: limit lower=0.0 upper=0.42249866384783047 effort=1000.0 velocity=1.0 -> lower=0.0 upper=0.43609180615466575 effort=1000.0 velocity=1.0; origin xyz=0.0 -0.2508016443505126 0.09227927174079907 rpy=0.0 -0.0 0.0 -> xyz=0.0 -0.2591924729349788 0.09227927174079907 rpy=0.0 -0.0 0.0
- joint drawer_0.496_0.183_0.557_object_28_world_fixed_joint: origin xyz=2.273771597051926 0.0 0.358505392213157 rpy=0.0 -0.0 0.0 -> xyz=2.2633274606463845 -0.008390828584466214 0.2817751122529999 rpy=0.0 -0.0 0.0
- joint drawer_0.537_0.207_0.480_object_33_world_fixed_joint: origin xyz=4.16187037873331 -1.0637107378191248 0.3326993390842733 rpy=0.0 -0.0 -1.5707963267948966 -> xyz=4.120093833111143 -1.0729040272980683 0.2559690591241162 rpy=0.0 -0.0 -1.5707963267948966
- joint drawer_0.590_0.193_0.517_object_32_world_fixed_joint: origin xyz=4.161870378733311 -0.565496920633376 0.3326993390842733 rpy=0.0 -0.0 -1.5707963267948966 -> xyz=4.120093833111144 -0.5746902101123195 0.2559690591241162 rpy=0.0 -0.0 -1.5707963267948966
- joint lower_left_cabinet_0.027_0.559_0.479_object_26_corpus_to_door_0_0: origin xyz=-0.24710690859287443 -0.28170623841306835 0.31863134815879773 rpy=0.0 -0.0 0.0 -> xyz=-0.24710690859287443 -0.28170623841306835 0.280254362563199 rpy=0.0 -0.0 0.0
- joint lower_left_cabinet_0.027_0.559_0.479_object_26_world_fixed_joint: origin xyz=4.16187037873331 -0.565496920633376 -0.3045633572333222 rpy=0.0 -0.0 -1.5707963267948966 -> xyz=4.120093833111143 -0.5746902101123195 -0.3045633572333221 rpy=0.0 -0.0 -1.5707963267948966
- joint lower_left_cabinet_0.410_0.554_0.009_object_24_corpus_to_door_0_0: origin xyz=-0.20590020455647107 -0.2745958281955071 0.31863134815879773 rpy=0.0 -0.0 0.0 -> xyz=-0.20590020455647107 -0.27919247293497884 0.280254362563199 rpy=0.0 -0.0 0.0
- joint lower_left_cabinet_0.410_0.554_0.009_object_24_world_fixed_joint: origin xyz=3.2184635266508304 -0.00379418384499447 -0.3045633572333222 rpy=0.0 -0.0 0.0 -> xyz=3.1766869810286638 -0.008390828584466214 -0.3045633572333221 rpy=0.0 -0.0 0.0
- joint lower_left_cabinet_0.470_0.567_0.015_object_22_corpus_to_door_0_0: origin xyz=-0.23315310527526945 -0.27919247293497884 0.31863134815879773 rpy=0.0 -0.0 0.0 -> xyz=-0.23315310527526945 -0.27919247293497884 0.280254362563199 rpy=0.0 -0.0 0.0
- joint lower_left_cabinet_0.477_0.710_0.022_object_1_corpus_to_door_0_0: origin xyz=-0.2363045883739352 -0.2708016443505126 0.31863134815879773 rpy=0.0 -0.0 0.0 -> xyz=-0.23441252064638118 -0.2708016443505126 0.35700833375439656 rpy=0.0 -0.0 0.0
- joint lower_left_cabinet_0.477_0.710_0.022_object_1_world_fixed_joint: origin xyz=-2.9526384500640894 0.0 -0.08358706587280118 rpy=0.0 -0.0 0.0 -> xyz=-2.956074050203862 0.0 -0.16034103706399883 rpy=0.0 -0.0 0.0
- joint lower_left_cabinet_0.481_0.705_0.014_object_5_corpus_to_door_0_0: origin xyz=-0.2383343788728849 -0.2708016443505126 0.31863134815879773 rpy=0.0 -0.0 0.0 -> xyz=-0.24359724168081093 -0.2708016443505126 0.35700833375439656 rpy=0.0 -0.0 0.0
- joint lower_left_cabinet_0.481_0.705_0.014_object_5_world_fixed_joint: origin xyz=-0.9646560651914683 0.0 -0.08358706587280118 rpy=0.0 -0.0 0.0 -> xyz=-0.9823889667232437 0.0 -0.16034103706399883 rpy=0.0 -0.0 0.0
- joint lower_left_cabinet_0.528_0.723_0.034_object_3_corpus_to_door_0_0: origin xyz=-0.261827898249521 -0.2708016443505126 0.31863134815879773 rpy=0.0 -0.0 0.0 -> xyz=-0.261827898249521 -0.2708016443505126 0.35700833375439656 rpy=0.0 -0.0 0.0
- joint lower_left_cabinet_0.528_0.723_0.034_object_3_world_fixed_joint: origin xyz=-1.9776809221478708 0.0 -0.08358706587280118 rpy=0.0 -0.0 0.0 -> xyz=-1.9830085900151975 0.0 -0.16034103706399883 rpy=0.0 -0.0 0.0
- joint lower_right_cabinet_0.016_0.561_0.478_object_27_corpus_to_door_0_0: origin xyz=0.24710690859287443 -0.28170623841306835 0.31863134815879773 rpy=0.0 -0.0 0.0 -> xyz=0.24710690859287443 -0.28170623841306835 0.280254362563199 rpy=0.0 -0.0 0.0
- joint lower_right_cabinet_0.016_0.561_0.478_object_27_world_fixed_joint: origin xyz=4.161870378733309 -1.063710737819125 -0.3045633572333222 rpy=0.0 -0.0 -1.5707963267948966 -> xyz=4.1200938331111425 -1.0729040272980686 -0.3045633572333221 rpy=0.0 -0.0 -1.5707963267948966
- joint lower_right_cabinet_0.398_0.559_0.010_object_25_corpus_to_door_0_0: origin xyz=0.20590020455647107 -0.2745958281955071 0.31863134815879773 rpy=0.0 -0.0 0.0 -> xyz=0.20590020455647107 -0.27919247293497884 0.280254362563199 rpy=0.0 -0.0 0.0
- joint lower_right_cabinet_0.398_0.559_0.010_object_25_world_fixed_joint: origin xyz=3.634263935763772 -0.00379418384499447 -0.3045633572333222 rpy=0.0 -0.0 0.0 -> xyz=3.5924873901416055 -0.008390828584466214 -0.3045633572333221 rpy=0.0 -0.0 0.0
- joint lower_right_cabinet_0.470_0.563_0.008_object_23_corpus_to_door_0_0: origin xyz=0.24359724168081093 -0.2708016443505126 0.31863134815879773 rpy=0.0 -0.0 0.0 -> xyz=0.23315310527526945 -0.27919247293497884 0.280254362563199 rpy=0.0 -0.0 0.0
- joint lower_right_cabinet_0.470_0.563_0.008_object_23_world_fixed_joint: origin xyz=2.764966080413548 0.0 -0.27875730410443844 rpy=0.0 -0.0 0.0 -> xyz=2.733633671196923 -0.008390828584466214 -0.27875730410443844 rpy=0.0 -0.0 0.0
- joint lower_right_cabinet_0.473_0.709_0.023_object_2_corpus_to_door_0_0: origin xyz=0.23441252064638118 -0.2708016443505126 0.31863134815879773 rpy=0.0 -0.0 0.0 -> xyz=0.23441252064638118 -0.2708016443505126 0.35700833375439656 rpy=0.0 -0.0 0.0
- joint lower_right_cabinet_0.473_0.709_0.023_object_2_world_fixed_joint: origin xyz=-2.477921341043773 0.0 -0.08358706587280118 rpy=0.0 -0.0 0.0 -> xyz=-2.4832490089110997 0.0 -0.16034103706399883 rpy=0.0 -0.0 0.0
- joint lower_right_cabinet_0.479_0.713_0.016_object_6_corpus_to_door_0_0: origin xyz=0.23736222231888626 -0.2708016443505126 0.31863134815879773 rpy=0.0 -0.0 0.0 -> xyz=0.24359724168081093 -0.2708016443505126 0.35700833375439656 rpy=0.0 -0.0 0.0
- joint lower_right_cabinet_0.479_0.713_0.016_object_6_world_fixed_joint: origin xyz=-0.48495946399969714 0.0 -0.08358706587280118 rpy=0.0 -0.0 0.0 -> xyz=-0.4911944833616218 0.0 -0.16034103706399883 rpy=0.0 -0.0 0.0
- joint lower_right_cabinet_0.509_0.725_0.023_object_4_corpus_to_door_0_0: origin xyz=0.25243128991699826 -0.2708016443505126 0.31863134815879773 rpy=0.0 -0.0 0.0 -> xyz=0.24359724168081093 -0.2708016443505126 0.35700833375439656 rpy=0.0 -0.0 0.0
- joint lower_right_cabinet_0.509_0.725_0.023_object_4_world_fixed_joint: origin xyz=-1.4594217339813516 0.0 -0.08358706587280118 rpy=0.0 -0.0 0.0 -> xyz=-1.4735834500848655 0.0 -0.16034103706399883 rpy=0.0 -0.0 0.0
- joint upper_left_cabinet_0.017_0.929_0.471_object_19_world_fixed_joint: origin xyz=4.228767027523136 -0.579342532468629 0.8417438520603431 rpy=0.0 -0.0 -1.5707963267948966 -> xyz=4.18699048190097 -0.5885358219475725 0.7266365865045872 rpy=0.0 -0.0 -1.5707963267948966
- joint upper_left_cabinet_0.279_0.929_0.299_object_18_world_fixed_joint: origin xyz=4.049086354776554 -0.08368340224450199 0.8417438520603431 rpy=0.0 -0.0 -0.7853981633974484 -> xyz=4.007309809154387 -0.09287669172344548 0.7266365865045871 rpy=0.0 -0.0 -0.7853981633974484
- joint upper_left_cabinet_0.392_0.934_0.031_object_12_corpus_to_door_0_0: origin xyz=-0.19522007790144802 -0.19872810015342557 0.4661418073058099 rpy=0.0 -0.0 0.0 -> xyz=-0.2002709616549837 -0.19872810015342557 0.4661418073058099 rpy=0.0 -0.0 0.0
- joint upper_left_cabinet_0.392_0.934_0.031_object_12_world_fixed_joint: origin xyz=1.4168850047422408 0.07207354419708706 0.870827707460851 rpy=0.0 -0.0 0.0 -> xyz=1.411834120988705 0.07207354419708706 0.7557204419050951 rpy=0.0 -0.0 0.0
- joint upper_left_cabinet_0.393_0.932_0.020_object_16_world_fixed_joint: origin xyz=3.178023727013106 0.07207354419708706 0.870827707460851 rpy=0.0 -0.0 0.0 -> xyz=3.1780111991027677 0.07207354419708706 0.7557204419050954 rpy=0.0 -0.0 0.0
- joint upper_left_cabinet_0.483_0.934_0.023_object_14_world_fixed_joint: origin xyz=2.257063785937655 0.07207354419708706 0.8708277074608513 rpy=0.0 -0.0 0.0 -> xyz=2.257063785937655 0.07207354419708706 0.7557204419050954 rpy=0.0 -0.0 0.0
- joint upper_right_cabinet_0.037_0.938_0.459_object_20_corpus_to_door_0_0: origin xyz=0.22864109689499956 -0.21480958962324118 0.4661418073058099 rpy=0.0 -0.0 0.0 -> xyz=0.23426129675762153 -0.21480958962324118 0.4661418073058099 rpy=0.0 -0.0 0.0
- joint upper_right_cabinet_0.037_0.938_0.459_object_20_world_fixed_joint: origin xyz=4.228767027523135 -1.04424492612125 0.8417438520603431 rpy=0.0 -0.0 -1.5707963267948966 -> xyz=4.186990481900969 -1.0590584154628155 0.7266365865045871 rpy=0.0 -0.0 -1.5707963267948966
- joint upper_right_cabinet_0.399_0.929_0.019_object_17_corpus_to_door_0_0: origin xyz=0.1985505308691463 -0.19872810015342557 0.4661418073058099 rpy=0.0 -0.0 0.0 -> xyz=0.19569707321311636 -0.19872810015342557 0.4661418073058099 rpy=0.0 -0.0 0.0
- joint upper_right_cabinet_0.399_0.929_0.019_object_17_world_fixed_joint: origin xyz=3.574271331095369 0.07207354419708706 0.870827707460851 rpy=0.0 -0.0 0.0 -> xyz=3.5714053455290005 0.07207354419708706 0.7557204419050954 rpy=0.0 -0.0 0.0
- joint upper_right_cabinet_0.403_0.935_0.022_object_13_world_fixed_joint: origin xyz=1.8143760442986725 0.07207354419708706 0.8708277074608513 rpy=0.0 -0.0 0.0 -> xyz=1.8143760442986725 0.07207354419708706 0.7557204419050952 rpy=0.0 -0.0 0.0
- joint upper_right_cabinet_0.483_0.931_0.019_object_15_corpus_to_door_0_0: origin xyz=0.24042304393916814 -0.19872810015342557 0.4661418073058099 rpy=0.0 -0.0 0.0 -> xyz=0.2404167799839988 -0.19872810015342557 0.4661418073058099 rpy=0.0 -0.0 0.0
- joint upper_right_cabinet_0.483_0.931_0.019_object_15_world_fixed_joint: origin xyz=2.739903609860822 0.07207354419708706 0.870827707460851 rpy=0.0 -0.0 0.0 -> xyz=2.7398973459056526 0.07207354419708706 0.7557204419050954 rpy=0.0 -0.0 0.0
