Commit message: working on heuristic update

File: simple_urdf_scenes/second_floor_test/second_floor_test.urdf (robot description, URDF)
Before this commit: robot Scene, 108 links, 107 joints
Joints:
- joint upper_right_cabinet_0.485_0.805_0.485_object_29_world_fixed_joint: origin xyz=6.3321385653473055 -1.4458530318084521 0.7045451622127326 rpy=0.0 -0.0 -1.5707963267948966 -> xyz=6.3321385653473055 -1.4458530318084524 0.7045451622127326 rpy=0.0 -0.0 -1.5707963267948966
