Commit message: working countertops and closed assets heuristic

File: simple_urdf_scenes/second_floor_test_2/second_floor_test_2.urdf (robot description, URDF)
Before this commit: robot Scene, 110 links, 109 joints
Links:
- added link counter_7.157_0.346_1.316_object_32_0, mass 0.1721196202767532; collision box size=6.691471370073138 0.6430559542051508 0.04; visual box size=6.691471370073138 0.6430559542051508 0.04
- added link counter_7.157_0.346_1.316_object_32_2, mass 0.018299642397866234; collision box size=0.711432740735816 0.6430559542051508 0.04; visual box size=0.711432740735816 0.6430559542051508 0.04
- link box_0.681_0.779_0.035_object_1: mass 0.3712258797535107 -> 0.3410271604722006; geometry collision box size=0.6805576078862803 0.6430559542051508 0.7792473101715351; visual box size=0.6805576078862803 0.6430559542051508 0.7792473101715351
- link box_23_to_26: mass 0.33978998703191204 -> 0.2877754213926684; geometry collision box size=0.6670559542051508 0.6430559542051508 0.6708766395076823; visual box size=0.6670559542051508 0.6430559542051508 0.6708766395076823
- link box_24_to_28: mass 0.09944137856639486 -> 0.08453220796710231; geometry collision box size=0.6670559542051508 0.6430559542051508 0.19706576516050908; visual box size=0.6670559542051508 0.6430559542051508 0.19706576516050908
- link box_26_to_23: mass 0.34021852010488196 -> 0.2879601385295633; geometry collision box size=0.6670559542051508 0.6430559542051508 0.6713072614539898; visual box size=0.6670559542051508 0.6430559542051508 0.6713072614539898
- link box_28_to_24: mass 0.10115834649853855 -> 0.08562018158847061; geometry collision box size=0.6670559542051508 0.6430559542051508 0.19960210437754258; visual box size=0.6670559542051508 0.6430559542051508 0.19960210437754258
- link drawer_0.347_0.159_0.022_object_27_corpus: mass 0.013683869358725082 -> 0.012601207079003371; geometry collision box size=0.02 0.6030559542051508 0.13960210437754259; collision box size=0.02 0.6030559542051508 0.13960210437754259
- link drawer_0.347_0.159_0.022_object_27_drawer_0_0: mass 0.09999999999999999 -> 0.09999999999999998; geometry collision box size=0.005 0.5357503587846357 0.10960210437754257; collision box size=0.005 0.5357503587846357 0.10960210437754257
- link drawer_0.356_0.160_0.012_object_28_corpus: mass 0.013683869358725082 -> 0.012601207079003371; geometry collision box size=0.02 0.6030559542051508 0.13960210437754259; collision box size=0.02 0.6030559542051508 0.13960210437754259
- link drawer_0.356_0.160_0.012_object_28_drawer_0_0: mass 0.09999999999999999 -> 0.09999999999999998; geometry collision box size=0.005 0.5357503587846357 0.10960210437754257; collision box size=0.005 0.5357503587846357 0.10960210437754257
- link drawer_0.463_0.157_0.017_object_22_corpus: mass 0.016737021082403825 -> 0.015417769072690157; geometry collision box size=0.02 0.6030559542051508 0.13621424342224722; collision box size=0.02 0.6030559542051508 0.13621424342224722
- link drawer_0.463_0.157_0.017_object_22_drawer_0_0: mass 0.10000000000000005 -> 0.10000000000000002; geometry collision box size=0.005 0.5357503587846357 0.10621424342224721; collision box size=0.005 0.5357503587846357 0.10621424342224721
- link drawer_0.465_0.158_0.021_object_5_corpus: mass 0.016955657742540667 -> 0.015620814346351099; geometry collision box size=0.02 0.6030559542051508 0.13887413043201827; collision box size=0.02 0.6030559542051508 0.13887413043201827
- link drawer_0.465_0.158_0.021_object_5_drawer_0_0: geometry collision box size=0.005 0.5357503587846357 0.10887413043201825; collision box size=0.005 0.5357503587846357 0.10887413043201825
- link drawer_0.465_0.161_0.025_object_3_corpus: mass 0.016955657742540667 -> 0.015696495390595533; geometry collision box size=0.02 0.6030559542051508 0.141135600878972; collision box size=0.02 0.6030559542051508 0.141135600878972
- link drawer_0.465_0.161_0.025_object_3_drawer_0_0: mass 0.1 -> 0.09999999999999999; geometry collision box size=0.005 0.5357503587846357 0.111135600878972; collision box size=0.005 0.5357503587846357 0.111135600878972
- link drawer_0.466_0.157_0.020_object_24_corpus: mass 0.016737021082403825 -> 0.015446194324906619; geometry collision box size=0.02 0.6030559542051508 0.13706576516050908; collision box size=0.02 0.6030559542051508 0.13706576516050908
- link drawer_0.466_0.157_0.020_object_24_drawer_0_0: mass 0.10000000000000005 -> 0.1; geometry collision box size=0.005 0.5357503587846357 0.10706576516050907; collision box size=0.005 0.5357503587846357 0.10706576516050907
- link drawer_0.467_0.159_0.022_object_9_corpus: mass 0.016955657742540667 -> 0.015620814346351099; geometry collision box size=0.02 0.6030559542051508 0.13887413043201827; collision box size=0.02 0.6030559542051508 0.13887413043201827
- link drawer_0.467_0.159_0.022_object_9_drawer_0_0: geometry collision box size=0.005 0.5357503587846357 0.10887413043201825; collision box size=0.005 0.5357503587846357 0.10887413043201825
- link drawer_0.468_0.159_0.024_object_7_corpus: mass 0.016955657742540667 -> 0.015620814346351099; geometry collision box size=0.02 0.6030559542051508 0.13887413043201827; collision box size=0.02 0.6030559542051508 0.13887413043201827
- link drawer_0.468_0.159_0.024_object_7_drawer_0_0: geometry collision box size=0.005 0.5357503587846357 0.10887413043201825; collision box size=0.005 0.5357503587846357 0.10887413043201825
- link drawer_0.469_0.159_0.023_object_15_corpus: mass 0.016960116998317974 -> 0.015579729275932399; geometry collision box size=0.02 0.6030559542051508 0.13764644292465758; collision box size=0.02 0.6030559542051508 0.13764644292465758
- link drawer_0.469_0.159_0.023_object_15_drawer_0_0: geometry collision box size=0.005 0.5357503587846357 0.10764644292465757; collision box size=0.005 0.5357503587846357 0.10764644292465757
- link drawer_0.470_0.158_0.022_object_11_corpus: mass 0.016955657742540667 -> 0.015598851667360098; geometry collision box size=0.02 0.6030559542051508 0.13821785051450466; collision box size=0.02 0.6030559542051508 0.13821785051450466
- link drawer_0.470_0.158_0.022_object_11_drawer_0_0: mass 0.1 -> 0.10000000000000002; geometry collision box size=0.005 0.5357503587846357 0.10821785051450465; collision box size=0.005 0.5357503587846357 0.10821785051450465
- link drawer_0.474_0.158_0.018_object_17_corpus: mass 0.01691177629237633 -> 0.015579729275932399; geometry collision box size=0.02 0.6030559542051508 0.13764644292465758; collision box size=0.02 0.6030559542051508 0.13764644292465758
- link drawer_0.474_0.158_0.018_object_17_drawer_0_0: mass 0.10000000000000002 -> 0.1; geometry collision box size=0.005 0.5357503587846357 0.10764644292465757; collision box size=0.005 0.5357503587846357 0.10764644292465757
- link drawer_0.474_0.296_0.034_object_12_corpus: mass 0.021873194785263422 -> 0.020224977493425736; geometry collision box size=0.02 0.6030559542051508 0.27645387703849544; collision box size=0.02 0.6030559542051508 0.27645387703849544
- link drawer_0.474_0.296_0.034_object_12_drawer_0_0: mass 0.1 -> 0.09999999999999999; geometry collision box size=0.005 0.5357503587846357 0.24645387703849547; collision box size=0.005 0.5357503587846357 0.24645387703849547
- link drawer_0.480_0.295_0.033_object_13_corpus: mass 0.021873194785263422 -> 0.020224977493425736; geometry collision box size=0.02 0.6030559542051508 0.27645387703849544; collision box size=0.02 0.6030559542051508 0.27645387703849544
- link drawer_0.480_0.295_0.033_object_13_drawer_0_0: mass 0.1 -> 0.09999999999999999; geometry collision box size=0.005 0.5357503587846357 0.24645387703849547; collision box size=0.005 0.5357503587846357 0.24645387703849547
- link lower_left_cabinet_0.350_0.626_0.016_object_25_corpus: mass 0.03138397630865971 -> 0.029060183535162744; geometry collision box size=0.02 0.6030559542051508 0.6055633846292184; collision box size=0.02 0.6030559542051508 0.6055633846292184
- link lower_left_cabinet_0.465_0.630_0.016_object_20_corpus: mass 0.03652870797346598 -> 0.03388287579439772; geometry collision box size=0.02 0.6030559542051508 0.6097460436711656; collision box size=0.02 0.6030559542051508 0.6097460436711656
- link lower_left_cabinet_0.468_0.628_0.018_object_16_corpus: mass 0.03658481941632824 -> 0.033935509624136176; geometry collision box size=0.02 0.6030559542051508 0.6091712833616468; collision box size=0.02 0.6030559542051508 0.6091712833616468
- link lower_left_cabinet_0.472_0.626_0.024_object_10_corpus: mass 0.036456653291617167 -> 0.03375978751922645; geometry collision box size=0.02 0.6030559542051508 0.6039204262798344; collision box size=0.02 0.6030559542051508 0.6039204262798344
- link lower_left_cabinet_0.472_0.626_0.024_object_10_door_0_0: mass 0.10000000000000003 -> 0.09999999999999999; geometry collision box size=0.013999999999999999 0.04 0.024; collision box size=0.013999999999999999 0.04 0.024
- link lower_left_cabinet_0.472_0.627_0.029_object_6_corpus: mass 0.036493551084897574 -> 0.03385005743853649; geometry collision box size=0.02 0.6030559542051508 0.6066178356087703; collision box size=0.02 0.6030559542051508 0.6066178356087703
- link lower_left_cabinet_0.477_0.630_0.023_object_23_corpus: mass 0.03644006089199226 -> 0.03381357940317814; geometry collision box size=0.02 0.6030559542051508 0.6108766395076822; collision box size=0.02 0.6030559542051508 0.6108766395076822
- link lower_left_cabinet_0.477_0.630_0.023_object_23_door_0_0: mass 0.09999999999999999 -> 0.1; geometry collision box size=0.013999999999999999 0.04 0.024; collision box size=0.013999999999999999 0.04 0.024
- link lower_right_cabinet_0.359_0.631_0.017_object_26_corpus: mass 0.03173422805395336 -> 0.029387508071138217; geometry collision box size=0.02 0.6030559542051508 0.6113072614539897; collision box size=0.02 0.6030559542051508 0.6113072614539897
- link lower_right_cabinet_0.466_0.627_0.027_object_4_corpus: mass 0.03652330505897709 -> 0.033877915317337554; geometry collision box size=0.02 0.6030559542051508 0.6074502735098642; collision box size=0.02 0.6030559542051508 0.6074502735098642
- link lower_right_cabinet_0.467_0.624_0.023_object_8_corpus: mass 0.03639713710957336 -> 0.03375978751922645; geometry collision box size=0.02 0.6030559542051508 0.6039204262798344; collision box size=0.02 0.6030559542051508 0.6039204262798344
- link lower_right_cabinet_0.467_0.629_0.016_object_18_corpus: mass 0.03658481941632824 -> 0.033935509624136176; geometry collision box size=0.02 0.6030559542051508 0.6091712833616468; collision box size=0.02 0.6030559542051508 0.6091712833616468
- link lower_right_cabinet_0.468_0.631_0.019_object_21_corpus: mass 0.03645485759379905 -> 0.03381357940317814; geometry collision box size=0.02 0.6030559542051508 0.6108766395076822; collision box size=0.02 0.6030559542051508 0.6108766395076822
- link lower_right_cabinet_0.469_0.629_0.024_object_14_corpus: mass 0.03658481941632824 -> 0.033935509624136176; geometry collision box size=0.02 0.6030559542051508 0.6091712833616468; collision box size=0.02 0.6030559542051508 0.6091712833616468
- link lower_right_cabinet_0.472_0.633_0.033_object_2_corpus: mass 0.03670784721755765 -> 0.033877915317337554; geometry collision box size=0.02 0.6030559542051508 0.6074502735098642; collision box size=0.02 0.6030559542051508 0.6074502735098642
- link lower_right_cabinet_0.472_0.633_0.033_object_2_door_0_0: mass 0.1 -> 0.10000000000000002; geometry collision box size=0.013999999999999999 0.04 0.024; collision box size=0.013999999999999999 0.04 0.024
- link sink_0.881_0.156_0.018_object_19_corpus: mass 0.04702122541269979 -> 0.04377527735886212; geometry collision box size=0.02 0.6030559542051508 0.15621424342224724; collision box size=0.02 0.6030559542051508 0.15621424342224724
- link upper_left_cabinet_0.439_0.774_0.054_object_29_corpus: mass 0.015298570972720164 -> 0.013662146006028733; geometry collision box size=0.01 0.31815440305646026 0.7642174125784422; collision box size=0.01 0.31815440305646026 0.7642174125784422
- link upper_left_cabinet_0.448_0.779_0.036_object_36_corpus: mass 0.012761431349739085 -> 0.012454972145307393; geometry collision box size=0.01 0.26756849542057215 0.7674330298635206; collision box size=0.01 0.26756849542057215 0.7674330298635206
- link upper_left_cabinet_0.461_0.777_0.042_object_34_corpus: mass 0.012266047429542938 -> 0.012454972145307393; geometry collision box size=0.01 0.26756849542057215 0.7674330298635206; collision box size=0.01 0.26756849542057215 0.7674330298635206
- link upper_left_cabinet_0.467_0.784_0.037_object_33_corpus: mass 0.011660813867311852 -> 0.011526846108040953; geometry collision box size=0.01 0.23958648613535363 0.7674330298635206; collision box size=0.01 0.23958648613535363 0.7674330298635206
- link upper_right_cabinet_0.439_0.776_0.032_object_30_corpus: mass 0.015298570972720164 -> 0.013662146006028733; geometry collision box size=0.01 0.31815440305646026 0.7642174125784422; collision box size=0.01 0.31815440305646026 0.7642174125784422
- link upper_right_cabinet_0.461_0.784_0.025_object_37_corpus: mass 0.013592124418274107 -> 0.013047435464421322; geometry collision box size=0.01 0.28543063206035924 0.7674330298635206; collision box size=0.01 0.28543063206035924 0.7674330298635206
- link upper_right_cabinet_0.464_0.781_0.032_object_35_corpus: mass 0.012761431349739085 -> 0.012454972145307393; geometry collision box size=0.01 0.26756849542057215 0.7674330298635206; collision box size=0.01 0.26756849542057215 0.7674330298635206
- link upper_right_cabinet_0.480_0.781_0.039_object_31_corpus: mass 0.01622480759928264 -> 0.014504829672714463; geometry collision box size=0.01 0.31815440305646026 0.7642174125784422; collision box size=0.01 0.31815440305646026 0.7642174125784422
Joints:
- added joint counter_7.157_0.346_1.316_object_32_0_world_fixed_joint: type fixed, parent world, child counter_7.157_0.346_1.316_object_32_0, origin xyz=-1.0301223473440464 0.0 0.18231662224232145 rpy=0.0 -0.0 0.0
- added joint counter_7.157_0.346_1.316_object_32_2_world_fixed_joint: type fixed, parent world, child counter_7.157_0.346_1.316_object_32_2, origin xyz=-4.735386009483191 -0.7152443474704833 0.18485296145935495 rpy=0.0 -0.0 1.5707963267948966
- joint box_0.681_0.779_0.035_object_1_world_fixed_joint: origin xyz=1.9753345349148619 0.0 -0.23074952465374932 rpy=0.0 -0.0 0.0 -> xyz=1.9753345349148619 0.0 -0.2378266184240967 rpy=0.0 -0.0 0.0
- joint box_23_to_26_world_fixed_joint: origin xyz=-4.737858032380616 0.0 -0.2916450965886376 rpy=0.0 -0.0 0.0 -> xyz=-4.709386009483191 0.0 -0.2901874626720287 rpy=0.0 -0.0 0.0
- joint box_24_to_28_world_fixed_joint: origin xyz=-4.737858032380616 0.0 0.10169287262831876 rpy=0.0 -0.0 0.0 -> xyz=-4.709386009483191 0.0 0.10378373966206693 rpy=0.0 -0.0 0.0
- joint box_26_to_23_world_fixed_joint: origin xyz=-4.7638580323806154 -0.025999999999999912 -0.29122231336747545 rpy=0.0 -0.0 1.5707963267948966 -> xyz=-4.735386009483191 -0.025999999999999912 -0.28997215169887497 rpy=0.0 -0.0 1.5707963267948966
- joint box_28_to_24_world_fixed_joint: origin xyz=-4.7638580323806154 -0.025999999999999912 0.10338680310596644 rpy=0.0 -0.0 1.5707963267948966 -> xyz=-4.735386009483191 -0.025999999999999912 0.10505190927058368 rpy=0.0 -0.0 1.5707963267948966
- joint drawer_0.347_0.159_0.022_object_27_corpus_to_drawer_0_0: limit lower=0.0 upper=0.5508 effort=1000.0 velocity=1.0 -> lower=0.0 upper=0.5046753229061722 effort=1000.0 velocity=1.0; origin xyz=0.0 -0.32999999999999996 0.0798010521887713 rpy=0.0 -0.0 0.0 -> xyz=0.0 -0.3015279771025754 0.0798010521887713 rpy=0.0 -0.0 0.0
- joint drawer_0.347_0.159_0.022_object_27_world_fixed_joint: origin xyz=-4.7638580323806154 -0.921574555551862 0.003585750917195152 rpy=0.0 -0.0 1.5707963267948966 -> xyz=-4.735386009483191 -0.8931025326544373 0.005250857081812388 rpy=0.0 -0.0 1.5707963267948966
- joint drawer_0.356_0.160_0.012_object_28_corpus_to_drawer_0_0: limit lower=0.0 upper=0.5508 effort=1000.0 velocity=1.0 -> lower=0.0 upper=0.5046753229061722 effort=1000.0 velocity=1.0; origin xyz=0.0 -0.32999999999999996 0.0798010521887713 rpy=0.0 -0.0 0.0 -> xyz=0.0 -0.3015279771025754 0.0798010521887713 rpy=0.0 -0.0 0.0
- joint drawer_0.356_0.160_0.012_object_28_world_fixed_joint: origin xyz=-4.7638580323806154 -0.5658581851839539 0.003585750917195152 rpy=0.0 -0.0 1.5707963267948966 -> xyz=-4.735386009483191 -0.5373861622865294 0.005250857081812388 rpy=0.0 -0.0 1.5707963267948966
- joint drawer_0.463_0.157_0.017_object_22_corpus_to_drawer_0_0: limit lower=0.0 upper=0.5508 effort=1000.0 velocity=1.0 -> lower=0.0 upper=0.5046753229061722 effort=1000.0 velocity=1.0; origin xyz=0.0 -0.32999999999999996 0.07810712171112362 rpy=0.0 -0.0 0.0 -> xyz=0.0 -0.3015279771025754 0.07810712171112362 rpy=0.0 -0.0 0.0
- joint drawer_0.463_0.157_0.017_object_22_world_fixed_joint: origin xyz=-3.6813976017403975 0.0 0.003585750917195152 rpy=0.0 -0.0 0.0 -> xyz=-3.6813976017403975 0.0 0.005250857081812388 rpy=0.0 -0.0 0.0
- joint drawer_0.465_0.158_0.021_object_5_corpus_to_drawer_0_0: limit lower=0.0 upper=0.5508 effort=1000.0 velocity=1.0 -> lower=0.0 upper=0.5046753229061722 effort=1000.0 velocity=1.0; origin xyz=0.0 -0.32999999999999996 0.07943706521600914 rpy=0.0 -0.0 0.0 -> xyz=0.0 -0.3015279771025754 0.07943706521600914 rpy=0.0 -0.0 0.0
- joint drawer_0.465_0.161_0.025_object_3_corpus_to_drawer_0_0: limit lower=0.0 upper=0.5508 effort=1000.0 velocity=1.0 -> lower=0.0 upper=0.5046753229061722 effort=1000.0 velocity=1.0; origin xyz=0.0 -0.32999999999999996 0.07943706521600914 rpy=0.0 -0.0 0.0 -> xyz=0.0 -0.3015279771025754 0.08056780043948601 rpy=0.0 -0.0 0.0
- joint drawer_0.466_0.157_0.020_object_24_corpus_to_drawer_0_0: limit lower=0.0 upper=0.5508 effort=1000.0 velocity=1.0 -> lower=0.0 upper=0.5046753229061722 effort=1000.0 velocity=1.0; origin xyz=0.0 -0.32999999999999996 0.07810712171112362 rpy=0.0 -0.0 0.0 -> xyz=0.0 -0.3015279771025754 0.07853288258025455 rpy=0.0 -0.0 0.0
- joint drawer_0.466_0.157_0.020_object_24_world_fixed_joint: origin xyz=-4.1443712221672095 0.0 0.003585750917195152 rpy=0.0 -0.0 0.0 -> xyz=-4.1443712221672095 0.0 0.005250857081812388 rpy=0.0 -0.0 0.0
- joint drawer_0.467_0.159_0.022_object_9_corpus_to_drawer_0_0: limit lower=0.0 upper=0.5508 effort=1000.0 velocity=1.0 -> lower=0.0 upper=0.5046753229061722 effort=1000.0 velocity=1.0; origin xyz=0.0 -0.32999999999999996 0.07943706521600914 rpy=0.0 -0.0 0.0 -> xyz=0.0 -0.3015279771025754 0.07943706521600914 rpy=0.0 -0.0 0.0
- joint drawer_0.468_0.159_0.024_object_7_corpus_to_drawer_0_0: limit lower=0.0 upper=0.5508 effort=1000.0 velocity=1.0 -> lower=0.0 upper=0.5046753229061722 effort=1000.0 velocity=1.0; origin xyz=0.0 -0.32999999999999996 0.07943706521600914 rpy=0.0 -0.0 0.0 -> xyz=0.0 -0.3015279771025754 0.07943706521600914 rpy=0.0 -0.0 0.0
- joint drawer_0.469_0.159_0.023_object_15_corpus_to_drawer_0_0: limit lower=0.0 upper=0.5508 effort=1000.0 velocity=1.0 -> lower=0.0 upper=0.5046753229061722 effort=1000.0 velocity=1.0; origin xyz=0.0 -0.32999999999999996 0.07949944433736249 rpy=0.0 -0.0 0.0 -> xyz=0.0 -0.3015279771025754 0.0788232214623288 rpy=0.0 -0.0 0.0
- joint drawer_0.469_0.159_0.023_object_15_world_fixed_joint: origin xyz=-1.8686351211105392 0.0 0.003585750917195152 rpy=0.0 -0.0 0.0 -> xyz=-1.8686351211105392 0.0 0.005250857081812388 rpy=0.0 -0.0 0.0
- joint drawer_0.470_0.158_0.022_object_11_corpus_to_drawer_0_0: limit lower=0.0 upper=0.5508 effort=1000.0 velocity=1.0 -> lower=0.0 upper=0.5046753229061722 effort=1000.0 velocity=1.0; origin xyz=0.0 -0.32999999999999996 0.07943706521600914 rpy=0.0 -0.0 0.0 -> xyz=0.0 -0.3015279771025754 0.07910892525725234 rpy=0.0 -0.0 0.0
- joint drawer_0.474_0.158_0.018_object_17_corpus_to_drawer_0_0: limit lower=0.0 upper=0.5508 effort=1000.0 velocity=1.0 -> lower=0.0 upper=0.5046753229061722 effort=1000.0 velocity=1.0; origin xyz=0.0 -0.32999999999999996 0.0788232214623288 rpy=0.0 -0.0 0.0 -> xyz=0.0 -0.3015279771025754 0.0788232214623288 rpy=0.0 -0.0 0.0
- joint drawer_0.474_0.158_0.018_object_17_world_fixed_joint: origin xyz=-2.335793901388174 0.0 0.003585750917195152 rpy=0.0 -0.0 0.0 -> xyz=-2.335793901388174 0.0 0.005250857081812388 rpy=0.0 -0.0 0.0
- joint drawer_0.474_0.296_0.034_object_12_corpus_to_drawer_0_0: limit lower=0.0 upper=0.5508 effort=1000.0 velocity=1.0 -> lower=0.0 upper=0.5046753229061722 effort=1000.0 velocity=1.0; origin xyz=0.0 -0.32999999999999996 0.1482269385192477 rpy=0.0 -0.0 0.0 -> xyz=0.0 -0.3015279771025754 0.1482269385192477 rpy=0.0 -0.0 0.0
- joint drawer_0.474_0.296_0.034_object_12_world_fixed_joint: origin xyz=-0.9343175605552694 0.0 -0.6255855324444517 rpy=0.0 -0.0 0.0 -> xyz=-0.9343175605552694 0.0 -0.6239204262798345 rpy=0.0 -0.0 0.0
- joint drawer_0.480_0.295_0.033_object_13_corpus_to_drawer_0_0: limit lower=0.0 upper=0.5508 effort=1000.0 velocity=1.0 -> lower=0.0 upper=0.5046753229061722 effort=1000.0 velocity=1.0; origin xyz=0.0 -0.32999999999999996 0.1482269385192477 rpy=0.0 -0.0 0.0 -> xyz=0.0 -0.3015279771025754 0.1482269385192477 rpy=0.0 -0.0 0.0
- joint drawer_0.480_0.295_0.033_object_13_world_fixed_joint: origin xyz=-1.4014763408329043 0.0 -0.6255855324444517 rpy=0.0 -0.0 0.0 -> xyz=-1.4014763408329043 0.0 -0.6239204262798345 rpy=0.0 -0.0 0.0
- joint lower_left_cabinet_0.350_0.626_0.016_object_25_corpus_to_door_0_0: origin xyz=-0.17585818518395402 -0.35 0.3127816923146092 rpy=0.0 -0.0 0.0 -> xyz=-0.17585818518395402 -0.3215279771025754 0.3127816923146092 rpy=0.0 -0.0 0.0
- joint lower_left_cabinet_0.350_0.626_0.016_object_25_world_fixed_joint: origin xyz=-4.7638580323806154 -0.921574555551862 -0.6219776337120233 rpy=0.0 -0.0 1.5707963267948966 -> xyz=-4.735386009483191 -0.8931025326544373 -0.6203125275474061 rpy=0.0 -0.0 1.5707963267948966
- joint lower_left_cabinet_0.465_0.630_0.016_object_20_corpus_to_door_0_0: origin xyz=-0.2307387789471751 -0.35 0.3148730218355828 rpy=0.0 -0.0 0.0 -> xyz=-0.2307387789471751 -0.3215279771025754 0.3148730218355828 rpy=0.0 -0.0 0.0
- joint lower_left_cabinet_0.465_0.630_0.016_object_20_world_fixed_joint: origin xyz=-3.2171720125798164 0.0 -0.6261602927539704 rpy=0.0 -0.0 0.0 -> xyz=-3.2171720125798164 0.0 -0.6244951865893532 rpy=0.0 -0.0 0.0
- joint lower_left_cabinet_0.468_0.628_0.018_object_16_corpus_to_door_0_0: origin xyz=-0.23157939013881734 -0.35 0.3145856416808234 rpy=0.0 -0.0 0.0 -> xyz=-0.23157939013881734 -0.3215279771025754 0.3145856416808234 rpy=0.0 -0.0 0.0
- joint lower_left_cabinet_0.468_0.628_0.018_object_16_world_fixed_joint: origin xyz=-2.335793901388174 0.0 -0.6255855324444517 rpy=0.0 -0.0 0.0 -> xyz=-2.335793901388174 0.0 -0.6239204262798345 rpy=0.0 -0.0 0.0
- joint lower_left_cabinet_0.472_0.626_0.024_object_10_corpus_to_door_0_0: origin xyz=-0.23157939013881734 -0.35 0.31279276622222585 rpy=0.0 -0.0 0.0 -> xyz=-0.23157939013881734 -0.3215279771025754 0.31196021313991723 rpy=0.0 -0.0 0.0
- joint lower_left_cabinet_0.472_0.626_0.024_object_10_world_fixed_joint: origin xyz=-0.4671587802776347 0.0 -0.6255855324444517 rpy=0.0 -0.0 0.0 -> xyz=-0.4671587802776347 0.0 -0.6239204262798345 rpy=0.0 -0.0 0.0
- joint lower_left_cabinet_0.472_0.627_0.029_object_6_corpus_to_door_0_0: origin xyz=-0.23157939013881734 -0.35 0.31330891780438513 rpy=0.0 -0.0 0.0 -> xyz=-0.23157939013881734 -0.3215279771025754 0.31330891780438513 rpy=0.0 -0.0 0.0
- joint lower_left_cabinet_0.477_0.630_0.023_object_23_corpus_to_door_0_0: origin xyz=-0.229486810213406 -0.35 0.31523084750583275 rpy=0.0 -0.0 0.0 -> xyz=-0.229486810213406 -0.3215279771025754 0.3154383197538411 rpy=0.0 -0.0 0.0
- joint lower_left_cabinet_0.477_0.630_0.023_object_23_world_fixed_joint: origin xyz=-4.1443712221672095 0.0 -0.6268759440944703 rpy=0.0 -0.0 0.0 -> xyz=-4.1443712221672095 0.0 -0.6256257824258699 rpy=0.0 -0.0 0.0
- joint lower_right_cabinet_0.359_0.631_0.017_object_26_corpus_to_door_0_0: origin xyz=0.17758690427701668 -0.35 0.31565363072699487 rpy=0.0 -0.0 0.0 -> xyz=0.17758690427701668 -0.3215279771025754 0.31565363072699487 rpy=0.0 -0.0 0.0
- joint lower_right_cabinet_0.359_0.631_0.017_object_26_world_fixed_joint: origin xyz=-4.7638580323806154 -0.5675869042770166 -0.6268759440944703 rpy=0.0 -0.0 1.5707963267948966 -> xyz=-4.735386009483191 -0.5391148813795921 -0.6256257824258699 rpy=0.0 -0.0 1.5707963267948966
- joint lower_right_cabinet_0.466_0.627_0.027_object_4_corpus_to_door_0_0: origin xyz=0.23157939013881734 -0.35 0.31372513675493213 rpy=0.0 -0.0 0.0 -> xyz=0.23157939013881734 -0.3215279771025754 0.31372513675493213 rpy=0.0 -0.0 0.0
- joint lower_right_cabinet_0.467_0.624_0.023_object_8_corpus_to_door_0_0: origin xyz=0.23157939013881734 -0.35 0.31196021313991723 rpy=0.0 -0.0 0.0 -> xyz=0.23157939013881734 -0.3215279771025754 0.31196021313991723 rpy=0.0 -0.0 0.0
- joint lower_right_cabinet_0.467_0.629_0.016_object_18_corpus_to_door_0_0: origin xyz=0.23157939013881734 -0.35 0.3145856416808234 rpy=0.0 -0.0 0.0 -> xyz=0.23157939013881734 -0.3215279771025754 0.3145856416808234 rpy=0.0 -0.0 0.0
- joint lower_right_cabinet_0.467_0.629_0.016_object_18_world_fixed_joint: origin xyz=-2.802952681665809 0.0 -0.6255855324444517 rpy=0.0 -0.0 0.0 -> xyz=-2.802952681665809 0.0 -0.6239204262798345 rpy=0.0 -0.0 0.0
- joint lower_right_cabinet_0.468_0.631_0.019_object_21_corpus_to_door_0_0: origin xyz=0.229486810213406 -0.35 0.3154383197538411 rpy=0.0 -0.0 0.0 -> xyz=0.229486810213406 -0.3215279771025754 0.3154383197538411 rpy=0.0 -0.0 0.0
- joint lower_right_cabinet_0.468_0.631_0.019_object_21_world_fixed_joint: origin xyz=-3.6813976017403975 0.0 -0.6272908885904871 rpy=0.0 -0.0 0.0 -> xyz=-3.6813976017403975 0.0 -0.6256257824258699 rpy=0.0 -0.0 0.0
- joint lower_right_cabinet_0.469_0.629_0.024_object_14_corpus_to_door_0_0: origin xyz=0.23157939013881734 -0.35 0.3145856416808234 rpy=0.0 -0.0 0.0 -> xyz=0.23157939013881734 -0.3215279771025754 0.3145856416808234 rpy=0.0 -0.0 0.0
- joint lower_right_cabinet_0.469_0.629_0.024_object_14_world_fixed_joint: origin xyz=-1.8686351211105392 0.0 -0.6255855324444517 rpy=0.0 -0.0 0.0 -> xyz=-1.8686351211105392 0.0 -0.6239204262798345 rpy=0.0 -0.0 0.0
- joint lower_right_cabinet_0.472_0.633_0.033_object_2_corpus_to_door_0_0: origin xyz=0.23157939013881734 -0.35 0.3163066387543221 rpy=0.0 -0.0 0.0 -> xyz=0.23157939013881734 -0.3215279771025754 0.31372513675493213 rpy=0.0 -0.0 0.0
- joint lower_right_cabinet_0.472_0.633_0.033_object_2_world_fixed_joint: origin xyz=1.4014763408329043 0.0 -0.6326132775086442 rpy=0.0 -0.0 0.0 -> xyz=1.4014763408329043 0.0 -0.6274502735098643 rpy=0.0 -0.0 0.0
- joint sink_0.881_0.156_0.018_object_19_world_fixed_joint: origin xyz=-3.0096420415269916 0.0 0.003585750917195152 rpy=0.0 -0.0 0.0 -> xyz=-3.0096420415269916 -2.8974245780410968e-09 0.005250857081812388 rpy=0.0 -0.0 0.0
- joint upper_left_cabinet_0.439_0.774_0.054_object_29_corpus_to_door_0_0: origin xyz=-0.21861359476534536 -0.19944542857812875 0.3871087062892211 rpy=0.0 -0.0 0.0 -> xyz=-0.21861359476534536 -0.17407720152823014 0.3871087062892211 rpy=0.0 -0.0 0.0
- joint upper_left_cabinet_0.439_0.774_0.054_object_29_world_fixed_joint: origin xyz=-4.914412603802487 -0.8798191459704706 0.7233759041720922 rpy=0.0 -0.0 1.5707963267948966 -> xyz=-4.8828367850575365 -0.8513471230730459 0.7326710267569503 rpy=0.0 -0.0 1.5707963267948966
- joint upper_left_cabinet_0.448_0.779_0.036_object_36_corpus_to_door_0_0: origin xyz=-0.22925011992319655 -0.15340395665046663 0.3887165149317603 rpy=0.0 -0.0 0.0 -> xyz=-0.22925011992319655 -0.1487842477102861 0.3887165149317603 rpy=0.0 -0.0 0.0
- joint upper_left_cabinet_0.448_0.779_0.036_object_36_world_fixed_joint: origin xyz=2.162209382207535 -0.8012505996159828 0.7048554973357577 rpy=0.0 -0.0 -1.5707963267948966 -> xyz=2.166829091147716 -0.8297226225134073 0.7166623934991525 rpy=0.0 -0.0 -1.5707963267948966
- joint upper_left_cabinet_0.461_0.777_0.042_object_34_corpus_to_door_0_0: origin xyz=-0.22925011992319655 -0.1459363084550216 0.3887165149317603 rpy=0.0 -0.0 0.0 -> xyz=-0.22925011992319655 -0.1487842477102861 0.3887165149317603 rpy=0.0 -0.0 0.0
- joint upper_left_cabinet_0.461_0.777_0.042_object_34_world_fixed_joint: origin xyz=2.1696770304029807 0.11974988007680343 0.7048554973357577 rpy=0.0 -0.0 -1.5707963267948966 -> xyz=2.166829091147716 0.09127785717937886 0.7166623934991526 rpy=0.0 -0.0 -1.5707963267948966
- joint upper_left_cabinet_0.467_0.784_0.037_object_33_corpus_to_door_0_0: origin xyz=-0.22925011992319655 -0.13681273553600526 0.3887165149317603 rpy=0.0 -0.0 0.0 -> xyz=-0.22925011992319655 -0.13479324306767682 0.3887165149317603 rpy=0.0 -0.0 0.0
- joint upper_left_cabinet_0.467_0.784_0.037_object_33_world_fixed_joint: origin xyz=2.1788006033219967 0.5802501199231965 0.7048554973357577 rpy=0.0 -0.0 -1.5707963267948966 -> xyz=2.180820095790325 0.551778097025772 0.7166623934991525 rpy=0.0 -0.0 -1.5707963267948966
- joint upper_right_cabinet_0.439_0.776_0.032_object_30_corpus_to_door_0_0: origin xyz=0.21861359476534536 -0.19944542857812875 0.3871087062892211 rpy=0.0 -0.0 0.0 -> xyz=0.21861359476534536 -0.17407720152823014 0.3871087062892211 rpy=0.0 -0.0 0.0
- joint upper_right_cabinet_0.439_0.776_0.032_object_30_world_fixed_joint: origin xyz=-4.914412603802487 -0.4405919564397799 0.7233759041720922 rpy=0.0 -0.0 1.5707963267948966 -> xyz=-4.8828367850575365 -0.4121199335423552 0.7326710267569503 rpy=0.0 -0.0 1.5707963267948966
- joint upper_right_cabinet_0.461_0.784_0.025_object_37_corpus_to_door_0_0: origin xyz=0.22925011992319655 -0.16592621129239776 0.3887165149317603 rpy=0.0 -0.0 0.0 -> xyz=0.22925011992319655 -0.15771531603017963 0.3887165149317603 rpy=0.0 -0.0 0.0
- joint upper_right_cabinet_0.461_0.784_0.025_object_37_world_fixed_joint: origin xyz=2.1496871275656035 -1.2617508394623758 0.7048554973357575 rpy=0.0 -0.0 -1.5707963267948966 -> xyz=2.1578980228278226 -1.2902228623598004 0.7166623934991525 rpy=0.0 -0.0 -1.5707963267948966
- joint upper_right_cabinet_0.464_0.781_0.032_object_35_corpus_to_door_0_0: origin xyz=0.22925011992319655 -0.15340395665046663 0.3887165149317603 rpy=0.0 -0.0 0.0 -> xyz=0.22925011992319655 -0.1487842477102861 0.3887165149317603 rpy=0.0 -0.0 0.0
- joint upper_right_cabinet_0.464_0.781_0.032_object_35_world_fixed_joint: origin xyz=2.1622093822075352 -0.3407503597695897 0.7048554973357577 rpy=0.0 -0.0 -1.5707963267948966 -> xyz=2.166829091147716 -0.36922238266701424 0.7166623934991525 rpy=0.0 -0.0 -1.5707963267948966
- joint upper_right_cabinet_0.480_0.781_0.039_object_31_corpus_to_door_0_0: origin xyz=0.23919863597467061 -0.19944542857812875 0.3871087062892211 rpy=0.0 -0.0 0.0 -> xyz=0.23919863597467061 -0.17407720152823014 0.3871087062892211 rpy=0.0 -0.0 0.0
- joint upper_right_cabinet_0.480_0.781_0.039_object_31_world_fixed_joint: origin xyz=-4.914412603802487 0.019220274300236095 0.7233759041720922 rpy=0.0 -0.0 1.5707963267948966 -> xyz=-4.8828367850575365 0.04769229719766077 0.7326710267569503 rpy=0.0 -0.0 1.5707963267948966
