Commit message: mesh pipeline (no clustering yet)

File: simple_urdf_scenes/basement_test_2/basement_test_2.urdf (robot description, URDF)
Before this commit: robot Scene, 151 links, 150 joints
Links:
- link box_0.310_0.842_0.981_object_26: mass 0.6202560509384899 -> 0.583872083293423; geometry collision box size=0.9807156973429858 0.7067464484576429 0.8423856292876121; visual box size=0.9807156973429858 0.7067464484576429 0.8423856292876121
- link box_0.602_0.725_0.043_object_35: mass 0.30905135235460923 -> 0.28981585335688237; geometry collision box size=0.6021619998788239 0.6635515409315338 0.7253274788229321; visual box size=0.6021619998788239 0.6635515409315338 0.7253274788229321
- link box_0.662_0.761_0.525_object_25: mass 0.2799124493371002 -> 0.26232525320836386; geometry collision box size=0.5246704664350093 0.6569003219439149 0.7611215306452649; visual box size=0.5246704664350093 0.6569003219439149 0.7611215306452649
- link box_19_to_21: mass 0.233357267974139 -> 0.2177842849147018; geometry collision box size=0.6159007144901296 0.5919007144901296 0.5974024043955687; visual box size=0.6159007144901296 0.5919007144901296 0.5974024043955687
- link box_20_to_22: mass 0.07712755561857769 -> 0.07198048594514879; geometry collision box size=0.6159007144901296 0.5919007144901296 0.1974491198482727; visual box size=0.6159007144901296 0.5919007144901296 0.1974491198482727
- link box_21_to_19: mass 0.23460923759426058 -> 0.21836183814107135; geometry collision box size=0.6159007144901296 0.5919007144901296 0.5989866862285518; visual box size=0.6159007144901296 0.5919007144901296 0.5989866862285518
- link box_22_to_20: mass 0.07775208936306312 -> 0.07236752195576229; geometry collision box size=0.6159007144901296 0.5919007144901296 0.19851079536548796; visual box size=0.6159007144901296 0.5919007144901296 0.19851079536548796
- link counter_0.697_0.200_3.231_object_42_2: mass 0.09158701306214269 -> 0.08588659504248548; geometry collision box size=3.2358675153520364 0.6635515409315338 0.04; visual box size=3.2358675153520364 0.6635515409315338 0.04
- link counter_3.084_0.217_2.078_object_43_2: mass 0.040801719843338476 -> 0.038238104502277485; geometry collision box size=1.4552475933153137 0.6569003219439149 0.04; visual box size=1.4552475933153137 0.6569003219439149 0.04
- link drawer_0.028_0.158_0.368_object_39_corpus: mass 0.01412544674538541 -> 0.013270167208939337; geometry collision box size=0.02 0.6235515409315338 0.13785832464574008; collision box size=0.02 0.6235515409315338 0.13785832464574008
- link drawer_0.028_0.158_0.368_object_39_drawer_0_0: mass 0.1 -> 0.09999999999999999; geometry collision box size=0.005 0.5541963868383804 0.10785832464574006; collision box size=0.005 0.5541963868383804 0.10785832464574006
- link drawer_0.365_0.159_0.022_object_41_corpus: mass 0.014220179975226767 -> 0.013359487452424873; geometry collision box size=0.02 0.6235515409315338 0.13856053701061374; collision box size=0.02 0.6235515409315338 0.13856053701061374
- link drawer_0.365_0.159_0.022_object_41_drawer_0_0: mass 0.10000000000000002 -> 0.09999999999999999; geometry collision box size=0.005 0.5541963868383804 0.10856053701061373; collision box size=0.005 0.5541963868383804 0.10856053701061373
- link drawer_0.461_0.155_0.011_object_29_corpus: mass 0.016002670961306246 -> 0.01498428250626202; geometry collision box size=0.02 0.586111661300921 0.13429078697326166; collision box size=0.02 0.586111661300921 0.13429078697326166
- link drawer_0.461_0.155_0.011_object_29_drawer_0_0: geometry collision box size=0.005 0.5205004951708289 0.10429078697326165; collision box size=0.005 0.5205004951708289 0.10429078697326165
- link drawer_0.463_0.154_0.012_object_28_corpus: mass 0.016002670961306246 -> 0.01498428250626202; geometry collision box size=0.02 0.586111661300921 0.13429078697326166; collision box size=0.02 0.586111661300921 0.13429078697326166
- link drawer_0.463_0.154_0.012_object_28_drawer_0_0: geometry collision box size=0.005 0.5205004951708289 0.10429078697326165; collision box size=0.005 0.5205004951708289 0.10429078697326165
- link drawer_0.463_0.248_0.017_object_30_corpus: mass 0.019190180222041102 -> 0.018008947222152426; geometry collision box size=0.02 0.586111661300921 0.22673021350256775; collision box size=0.02 0.586111661300921 0.22673021350256775
- link drawer_0.463_0.248_0.017_object_30_drawer_0_0: geometry collision box size=0.005 0.5205004951708289 0.19673021350256772; collision box size=0.005 0.5205004951708289 0.19673021350256772
- link drawer_0.464_0.154_0.014_object_32_corpus: mass 0.016002670961306246 -> 0.01498428250626202; geometry collision box size=0.02 0.586111661300921 0.13429078697326166; collision box size=0.02 0.586111661300921 0.13429078697326166
- link drawer_0.464_0.154_0.014_object_32_drawer_0_0: geometry collision box size=0.005 0.5205004951708289 0.10429078697326165; collision box size=0.005 0.5205004951708289 0.10429078697326165
- link drawer_0.464_0.154_0.017_object_27_corpus: mass 0.016002670961306246 -> 0.01498428250626202; geometry collision box size=0.02 0.586111661300921 0.13429078697326166; collision box size=0.02 0.586111661300921 0.13429078697326166
- link drawer_0.464_0.154_0.017_object_27_drawer_0_0: geometry collision box size=0.005 0.5205004951708289 0.10429078697326165; collision box size=0.005 0.5205004951708289 0.10429078697326165
- link drawer_0.465_0.159_0.014_object_22_corpus: mass 0.015391478017598341 -> 0.01436303653505577; geometry collision box size=0.02 0.5519007144901296 0.13851079536548797; collision box size=0.02 0.5519007144901296 0.13851079536548797
- link drawer_0.465_0.159_0.014_object_22_drawer_0_0: mass 0.1 -> 0.10000000000000002; geometry collision box size=0.005 0.48971064304111667 0.10851079536548795; collision box size=0.005 0.48971064304111667 0.10851079536548795
- link drawer_0.468_0.155_0.015_object_33_corpus: mass 0.016002670961306246 -> 0.01498428250626202; geometry collision box size=0.02 0.586111661300921 0.13429078697326166; collision box size=0.02 0.586111661300921 0.13429078697326166
- link drawer_0.468_0.155_0.015_object_33_drawer_0_0: geometry collision box size=0.005 0.5205004951708289 0.10429078697326165; collision box size=0.005 0.5205004951708289 0.10429078697326165
- link drawer_0.470_0.154_0.020_object_34_corpus: mass 0.016002670961306246 -> 0.01498428250626202; geometry collision box size=0.02 0.586111661300921 0.13429078697326166; collision box size=0.02 0.586111661300921 0.13429078697326166
- link drawer_0.470_0.154_0.020_object_34_drawer_0_0: geometry collision box size=0.005 0.5205004951708289 0.10429078697326165; collision box size=0.005 0.5205004951708289 0.10429078697326165
- link drawer_0.472_0.247_0.017_object_31_corpus: mass 0.019190180222041102 -> 0.018008947222152426; geometry collision box size=0.02 0.586111661300921 0.22673021350256775; collision box size=0.02 0.586111661300921 0.22673021350256775
- link drawer_0.472_0.247_0.017_object_31_drawer_0_0: geometry collision box size=0.005 0.5205004951708289 0.19673021350256772; collision box size=0.005 0.5205004951708289 0.19673021350256772
- link drawer_0.477_0.158_0.016_object_24_corpus: mass 0.015391478017598341 -> 0.01436303653505577; geometry collision box size=0.02 0.5519007144901296 0.13851079536548797; collision box size=0.02 0.5519007144901296 0.13851079536548797
- link drawer_0.477_0.158_0.016_object_24_drawer_0_0: mass 0.1 -> 0.10000000000000002; geometry collision box size=0.005 0.48971064304111667 0.10851079536548795; collision box size=0.005 0.48971064304111667 0.10851079536548795
- link lower_left_cabinet_0.370_0.563_0.023_object_38_corpus: mass 0.03021162013627085 -> 0.028493355108827403; geometry collision box size=0.02 0.6235515409315338 0.5428615187397526; collision box size=0.02 0.6235515409315338 0.5428615187397526
- link lower_left_cabinet_0.464_0.559_0.015_object_21_corpus: mass 0.031134596403209782 -> 0.02921682782042771; geometry collision box size=0.02 0.5519007144901296 0.5389866862285517; collision box size=0.02 0.5519007144901296 0.5389866862285517
- link lower_left_cabinet_0.484_0.717_0.027_object_36_corpus: mass 0.04122121507286721 -> 0.03896525917585969; geometry collision box size=0.02 0.6235515409315338 0.7053274788229321; collision box size=0.02 0.6235515409315338 0.7053274788229321
- link lower_right_cabinet_0.366_0.563_0.024_object_40_corpus: mass 0.03021162013627085 -> 0.028493355108827403; geometry collision box size=0.02 0.6235515409315338 0.5428615187397526; collision box size=0.02 0.6235515409315338 0.5428615187397526
- link lower_right_cabinet_0.474_0.719_0.027_object_37_corpus: mass 0.04122121507286721 -> 0.03896525917585969; geometry collision box size=0.02 0.6235515409315338 0.7053274788229321; collision box size=0.02 0.6235515409315338 0.7053274788229321
- link lower_right_cabinet_0.480_0.561_0.021_object_23_corpus: mass 0.031134596403209782 -> 0.02921682782042771; geometry collision box size=0.02 0.5519007144901296 0.5389866862285517; collision box size=0.02 0.5519007144901296 0.5389866862285517
- link upper_left_cabinet_0.469_0.936_0.030_object_52_corpus: mass 0.02105937507711232 -> 0.019443939017829866; geometry collision box size=0.01 0.4104104741203176 0.9259811505211948; collision box size=0.01 0.4104104741203176 0.9259811505211948
- link upper_right_cabinet_0.461_0.940_0.021_object_53_corpus: mass 0.02105937507711232 -> 0.019443939017829866; geometry collision box size=0.01 0.4104104741203176 0.9259811505211948; collision box size=0.01 0.4104104741203176 0.9259811505211948
Joints:
- joint box_0.310_0.842_0.981_object_26_world_fixed_joint: origin xyz=3.9758061229332213 -2.262207446563944 0.043267142651248036 rpy=0.0 -0.0 -1.5707963267948966 -> xyz=3.9537856833114944 -2.262207446563944 0.043267142651248036 rpy=0.0 -0.0 -1.5707963267948966
- joint box_0.602_0.725_0.043_object_35_world_fixed_joint: origin xyz=3.997403576696276 -3.981250147743884 0.05435983567663316 rpy=0.0 -0.0 -1.5707963267948966 -> xyz=3.975383137074549 -3.981250147743884 0.05435983567663316 rpy=0.0 -0.0 -1.5707963267948966
- joint box_0.662_0.761_0.525_object_25_world_fixed_joint: origin xyz=4.000729186190085 -1.5095143646749467 0.08389919197242163 rpy=0.0 -0.0 -1.5707963267948966 -> xyz=3.9787087465683584 -1.5095143646749467 0.08389919197242163 rpy=0.0 -0.0 -1.5707963267948966
- joint box_19_to_21_world_fixed_joint: origin xyz=4.007228989916978 0.017348352667927336 0.04724795973178181 rpy=0.0 -0.0 0.0 -> xyz=3.9852085502952512 0.017348352667927336 0.04724795973178181 rpy=0.0 -0.0 0.0
- joint box_20_to_22_world_fixed_joint: origin xyz=4.007228989916978 0.017348352667927336 0.4046737218537025 rpy=0.0 -0.0 0.0 -> xyz=3.9852085502952512 0.017348352667927336 0.4046737218537025 rpy=0.0 -0.0 0.0
- joint box_21_to_19_world_fixed_joint: origin xyz=4.033228989916978 -0.008651647332072687 0.048040100648273354 rpy=0.0 -0.0 -1.5707963267948966 -> xyz=4.011208550295251 -0.008651647332072687 0.048040100648273354 rpy=0.0 -0.0 -1.5707963267948966
- joint box_22_to_20_world_fixed_joint: origin xyz=4.033228989916978 -0.008651647332072576 0.4052045596123101 rpy=0.0 -0.0 -1.5707963267948966 -> xyz=4.011208550295251 -0.008651647332072576 0.4052045596123101 rpy=0.0 -0.0 -1.5707963267948966
- joint counter_0.697_0.200_3.231_object_42_2_world_fixed_joint: origin xyz=3.9974035766962768 -4.372869546205965 0.4331181520155335 rpy=0.0 -0.0 -1.5707963267948966 -> xyz=3.975383137074549 -4.372869546205965 0.4331181520155335 rpy=0.0 -0.0 -1.5707963267948966
- joint counter_3.084_0.217_2.078_object_43_2_world_fixed_joint: origin xyz=4.000729186190085 -1.0442258012347942 0.4844599572950541 rpy=0.0 -0.0 -1.5707963267948966 -> xyz=3.9787087465683584 -1.0442258012347942 0.4844599572950541 rpy=0.0 -0.0 -1.5707963267948966
- joint drawer_0.028_0.158_0.368_object_39_corpus_to_drawer_0_0: limit lower=0.0 upper=0.556949860341739 effort=1000.0 velocity=1.0 -> lower=0.0 upper=0.5212767481545424 effort=1000.0 velocity=1.0; origin xyz=0.0 -0.33379621008749316 0.07892916232287005 rpy=0.0 -0.0 0.0 -> xyz=0.0 -0.3117757704657669 0.07892916232287005 rpy=0.0 -0.0 0.0
- joint drawer_0.028_0.158_0.368_object_39_world_fixed_joint: origin xyz=3.9974035766962768 -5.434594983565735 0.2591652504423592 rpy=0.0 -0.0 -1.5707963267948966 -> xyz=3.975383137074549 -5.434594983565735 0.2591652504423592 rpy=0.0 -0.0 -1.5707963267948966
- joint drawer_0.365_0.159_0.022_object_41_corpus_to_drawer_0_0: limit lower=0.0 upper=0.556949860341739 effort=1000.0 velocity=1.0 -> lower=0.0 upper=0.5212767481545424 effort=1000.0 velocity=1.0; origin xyz=0.0 -0.33379621008749316 0.07928026850530688 rpy=0.0 -0.0 0.0 -> xyz=0.0 -0.3117757704657669 0.07928026850530688 rpy=0.0 -0.0 0.0
- joint drawer_0.365_0.159_0.022_object_41_world_fixed_joint: origin xyz=3.9974035766962768 -5.805795612658985 0.25455761500491975 rpy=0.0 -0.0 -1.5707963267948966 -> xyz=3.975383137074549 -5.805795612658985 0.25455761500491975 rpy=0.0 -0.0 -1.5707963267948966
- joint drawer_0.461_0.155_0.011_object_29_corpus_to_drawer_0_0: limit lower=0.0 upper=0.5266235578409426 effort=1000.0 velocity=1.0 -> lower=0.0 upper=0.490950445653746 effort=1000.0 velocity=1.0; origin xyz=0.0 -0.31507627027218676 0.07714539348663084 rpy=0.0 -0.0 0.0 -> xyz=0.0 -0.2930558306504605 0.07714539348663084 rpy=0.0 -0.0 0.0
- joint drawer_0.461_0.155_0.011_object_29_world_fixed_joint: origin xyz=4.016123516511582 -2.9844662583776955 -0.04584878583168572 rpy=0.0 -0.0 -1.5707963267948966 -> xyz=3.9941030768898553 -2.9844662583776955 -0.04584878583168572 rpy=0.0 -0.0 -1.5707963267948966
- joint drawer_0.463_0.154_0.012_object_28_corpus_to_drawer_0_0: limit lower=0.0 upper=0.5266235578409426 effort=1000.0 velocity=1.0 -> lower=0.0 upper=0.490950445653746 effort=1000.0 velocity=1.0; origin xyz=0.0 -0.31507627027218676 0.07714539348663084 rpy=0.0 -0.0 0.0 -> xyz=0.0 -0.2930558306504605 0.07714539348663084 rpy=0.0 -0.0 0.0
- joint drawer_0.463_0.154_0.012_object_28_world_fixed_joint: origin xyz=4.016123516511582 -2.984466258377696 0.10844200114157593 rpy=0.0 -0.0 -1.5707963267948966 -> xyz=3.9941030768898553 -2.984466258377696 0.10844200114157593 rpy=0.0 -0.0 -1.5707963267948966
- joint drawer_0.463_0.248_0.017_object_30_corpus_to_drawer_0_0: limit lower=0.0 upper=0.5266235578409426 effort=1000.0 velocity=1.0 -> lower=0.0 upper=0.490950445653746 effort=1000.0 velocity=1.0; origin xyz=0.0 -0.31507627027218676 0.12336510675128388 rpy=0.0 -0.0 0.0 -> xyz=0.0 -0.2930558306504605 0.12336510675128388 rpy=0.0 -0.0 0.0
- joint drawer_0.463_0.248_0.017_object_30_world_fixed_joint: origin xyz=4.016123516511582 -2.9844662583776955 -0.29257899933425346 rpy=0.0 -0.0 -1.5707963267948966 -> xyz=3.9941030768898553 -2.9844662583776955 -0.29257899933425346 rpy=0.0 -0.0 -1.5707963267948966
- joint drawer_0.464_0.154_0.014_object_32_corpus_to_drawer_0_0: limit lower=0.0 upper=0.5266235578409426 effort=1000.0 velocity=1.0 -> lower=0.0 upper=0.490950445653746 effort=1000.0 velocity=1.0; origin xyz=0.0 -0.31507627027218676 0.07714539348663084 rpy=0.0 -0.0 0.0 -> xyz=0.0 -0.2930558306504605 0.07714539348663084 rpy=0.0 -0.0 0.0
- joint drawer_0.464_0.154_0.014_object_32_world_fixed_joint: origin xyz=4.016123516511582 -3.448268184662213 -0.04584878583168572 rpy=0.0 -0.0 -1.5707963267948966 -> xyz=3.9941030768898553 -3.448268184662213 -0.04584878583168572 rpy=0.0 -0.0 -1.5707963267948966
- joint drawer_0.464_0.154_0.017_object_27_corpus_to_drawer_0_0: limit lower=0.0 upper=0.5266235578409426 effort=1000.0 velocity=1.0 -> lower=0.0 upper=0.490950445653746 effort=1000.0 velocity=1.0; origin xyz=0.0 -0.31507627027218676 0.07714539348663084 rpy=0.0 -0.0 0.0 -> xyz=0.0 -0.2930558306504605 0.07714539348663084 rpy=0.0 -0.0 0.0
- joint drawer_0.464_0.154_0.017_object_27_world_fixed_joint: origin xyz=4.016123516511582 -2.984466258377696 0.2627327881148376 rpy=0.0 -0.0 -1.5707963267948966 -> xyz=3.9941030768898553 -2.984466258377696 0.2627327881148376 rpy=0.0 -0.0 -1.5707963267948966
- joint drawer_0.465_0.159_0.014_object_22_corpus_to_drawer_0_0: limit lower=0.0 upper=0.49891269092420154 effort=1000.0 velocity=1.0 -> lower=0.0 upper=0.46323957873700505 effort=1000.0 velocity=1.0; origin xyz=0.0 -0.29797079686679107 0.07925539768274399 rpy=0.0 -0.0 0.0 -> xyz=0.0 -0.2759503572450648 0.07925539768274399 rpy=0.0 -0.0 0.0
- joint drawer_0.465_0.159_0.014_object_22_world_fixed_joint: origin xyz=4.033228989916978 -0.5492462862972135 0.3059491619295661 rpy=0.0 -0.0 -1.5707963267948966 -> xyz=4.011208550295251 -0.5492462862972135 0.3059491619295661 rpy=0.0 -0.0 -1.5707963267948966
- joint drawer_0.468_0.155_0.015_object_33_corpus_to_drawer_0_0: limit lower=0.0 upper=0.5266235578409426 effort=1000.0 velocity=1.0 -> lower=0.0 upper=0.490950445653746 effort=1000.0 velocity=1.0; origin xyz=0.0 -0.31507627027218676 0.07714539348663084 rpy=0.0 -0.0 0.0 -> xyz=0.0 -0.2930558306504605 0.07714539348663084 rpy=0.0 -0.0 0.0
- joint drawer_0.468_0.155_0.015_object_33_world_fixed_joint: origin xyz=4.016123516511582 -3.448268184662213 0.10844200114157593 rpy=0.0 -0.0 -1.5707963267948966 -> xyz=3.9941030768898553 -3.448268184662213 0.10844200114157593 rpy=0.0 -0.0 -1.5707963267948966
- joint drawer_0.470_0.154_0.020_object_34_corpus_to_drawer_0_0: limit lower=0.0 upper=0.5266235578409426 effort=1000.0 velocity=1.0 -> lower=0.0 upper=0.490950445653746 effort=1000.0 velocity=1.0; origin xyz=0.0 -0.31507627027218676 0.07714539348663084 rpy=0.0 -0.0 0.0 -> xyz=0.0 -0.2930558306504605 0.07714539348663084 rpy=0.0 -0.0 0.0
- joint drawer_0.470_0.154_0.020_object_34_world_fixed_joint: origin xyz=4.016123516511582 -3.4482681846622136 0.2627327881148376 rpy=0.0 -0.0 -1.5707963267948966 -> xyz=3.9941030768898553 -3.4482681846622136 0.2627327881148376 rpy=0.0 -0.0 -1.5707963267948966
- joint drawer_0.472_0.247_0.017_object_31_corpus_to_drawer_0_0: limit lower=0.0 upper=0.5266235578409426 effort=1000.0 velocity=1.0 -> lower=0.0 upper=0.490950445653746 effort=1000.0 velocity=1.0; origin xyz=0.0 -0.31507627027218676 0.12336510675128388 rpy=0.0 -0.0 0.0 -> xyz=0.0 -0.2930558306504605 0.12336510675128388 rpy=0.0 -0.0 0.0
- joint drawer_0.472_0.247_0.017_object_31_world_fixed_joint: origin xyz=4.016123516511582 -3.448268184662213 -0.29257899933425346 rpy=0.0 -0.0 -1.5707963267948966 -> xyz=3.9941030768898553 -3.448268184662213 -0.29257899933425346 rpy=0.0 -0.0 -1.5707963267948966
- joint drawer_0.477_0.158_0.016_object_24_corpus_to_drawer_0_0: limit lower=0.0 upper=0.49891269092420154 effort=1000.0 velocity=1.0 -> lower=0.0 upper=0.46323957873700505 effort=1000.0 velocity=1.0; origin xyz=0.0 -0.29797079686679107 0.07925539768274399 rpy=0.0 -0.0 0.0 -> xyz=0.0 -0.2759503572450648 0.07925539768274399 rpy=0.0 -0.0 0.0
- joint drawer_0.477_0.158_0.016_object_24_world_fixed_joint: origin xyz=4.033228989916978 -1.0145348497373659 0.3059491619295661 rpy=0.0 -0.0 -1.5707963267948966 -> xyz=4.011208550295251 -1.0145348497373659 0.3059491619295661 rpy=0.0 -0.0 -1.5707963267948966
- joint lower_left_cabinet_0.370_0.563_0.023_object_38_corpus_to_door_0_0: origin xyz=-0.18300769122299765 -0.3537962100874932 0.2814307593698763 rpy=0.0 -0.0 0.0 -> xyz=-0.18300769122299765 -0.3317757704657669 0.2814307593698763 rpy=0.0 -0.0 0.0
- joint lower_left_cabinet_0.370_0.563_0.023_object_38_world_fixed_joint: origin xyz=3.9974035766962768 -5.435780230212989 -0.3083039037348329 rpy=0.0 -0.0 -1.5707963267948966 -> xyz=3.975383137074549 -5.435780230212989 -0.3083039037348329 rpy=0.0 -0.0 -1.5707963267948966
- joint lower_left_cabinet_0.464_0.559_0.015_object_21_corpus_to_door_0_0: origin xyz=-0.2298572546539724 -0.3179707968667911 0.27949334311427587 rpy=0.0 -0.0 0.0 -> xyz=-0.2298572546539724 -0.2959503572450648 0.27949334311427587 rpy=0.0 -0.0 0.0
- joint lower_left_cabinet_0.464_0.559_0.015_object_21_world_fixed_joint: origin xyz=4.033228989916978 -0.5484592592311098 -0.25145324246600254 rpy=0.0 -0.0 -1.5707963267948966 -> xyz=4.011208550295251 -0.5484592592311098 -0.25145324246600254 rpy=0.0 -0.0 -1.5707963267948966
- joint lower_left_cabinet_0.484_0.717_0.027_object_36_corpus_to_door_0_0: origin xyz=-0.24011034782667395 -0.3537962100874932 0.36266373941146607 rpy=0.0 -0.0 0.0 -> xyz=-0.24011034782667395 -0.3317757704657669 0.36266373941146607 rpy=0.0 -0.0 0.0
- joint lower_left_cabinet_0.484_0.717_0.027_object_36_world_fixed_joint: origin xyz=3.9974035766962763 -4.524441495509969 -0.3083039037348329 rpy=0.0 -0.0 -1.5707963267948966 -> xyz=3.97538313707455 -4.524441495509969 -0.3083039037348329 rpy=0.0 -0.0 -1.5707963267948966
- joint lower_right_cabinet_0.366_0.563_0.024_object_40_corpus_to_door_0_0: origin xyz=0.18300769122299765 -0.3537962100874932 0.2814307593698763 rpy=0.0 -0.0 0.0 -> xyz=0.18300769122299765 -0.3317757704657669 0.2814307593698763 rpy=0.0 -0.0 0.0
- joint lower_right_cabinet_0.366_0.563_0.024_object_40_world_fixed_joint: origin xyz=3.9974035766962768 -5.805795612658985 -0.3083039037348329 rpy=0.0 -0.0 -1.5707963267948966 -> xyz=3.975383137074549 -5.805795612658985 -0.3083039037348329 rpy=0.0 -0.0 -1.5707963267948966
- joint lower_right_cabinet_0.474_0.719_0.027_object_37_corpus_to_door_0_0: origin xyz=0.24011034782667395 -0.3537962100874932 0.36266373941146607 rpy=0.0 -0.0 0.0 -> xyz=0.24011034782667395 -0.3317757704657669 0.36266373941146607 rpy=0.0 -0.0 0.0
- joint lower_right_cabinet_0.474_0.719_0.027_object_37_world_fixed_joint: origin xyz=3.9974035766962768 -5.008662191163317 -0.3083039037348329 rpy=0.0 -0.0 -1.5707963267948966 -> xyz=3.975383137074549 -5.008662191163317 -0.3083039037348329 rpy=0.0 -0.0 -1.5707963267948966
- joint lower_right_cabinet_0.480_0.561_0.021_object_23_corpus_to_door_0_0: origin xyz=0.2298572546539724 -0.3179707968667911 0.27949334311427587 rpy=0.0 -0.0 0.0 -> xyz=0.2298572546539724 -0.2959503572450648 0.27949334311427587 rpy=0.0 -0.0 0.0
- joint lower_right_cabinet_0.480_0.561_0.021_object_23_world_fixed_joint: origin xyz=4.033228989916978 -1.0121737685390548 -0.25145324246600254 rpy=0.0 -0.0 -1.5707963267948966 -> xyz=4.011208550295251 -1.0121737685390548 -0.25145324246600254 rpy=0.0 -0.0 -1.5707963267948966
- joint upper_left_cabinet_0.469_0.936_0.030_object_52_corpus_to_door_0_0: origin xyz=-0.2335094263516041 -0.2422256766818851 0.4679905752605974 rpy=0.0 -0.0 0.0 -> xyz=-0.2335094263516041 -0.22020523706015882 0.4679905752605974 rpy=0.0 -0.0 0.0
- joint upper_left_cabinet_0.469_0.936_0.030_object_52_world_fixed_joint: origin xyz=4.108974110101884 -0.5511114309287416 0.8624776351863548 rpy=0.0 -0.0 -1.5707963267948966 -> xyz=4.086953670480157 -0.5511114309287415 0.8624776351863548 rpy=0.0 -0.0 -1.5707963267948966
- joint upper_right_cabinet_0.461_0.940_0.021_object_53_corpus_to_door_0_0: origin xyz=0.2335094263516041 -0.2422256766818851 0.4679905752605974 rpy=0.0 -0.0 0.0 -> xyz=0.2335094263516041 -0.22020523706015882 0.4679905752605974 rpy=0.0 -0.0 0.0
- joint upper_right_cabinet_0.461_0.940_0.021_object_53_world_fixed_joint: origin xyz=4.108974110101884 -1.02013028363195 0.8624776351863548 rpy=0.0 -0.0 -1.5707963267948966 -> xyz=4.086953670480157 -1.0201302836319497 0.8624776351863548 rpy=0.0 -0.0 -1.5707963267948966
